File: data_logger.kicad_sch (KiCad schematic)
At the start: 30 parts, among them J2 Conn_01x04, Q2 MBT3904DW1, U1 Teensy4.1, U2 TJA1050T/CM,118, U2 XC6220B331, U5 LIS3DHTR, U7 ESP32-PICO-D4

Commit message: layout
Parts:
- added J2: I2C, symbol Connector_Generic:Conn_01x04
- added J3: SERIAL1, symbol Connector_Generic:Conn_01x04
- added J4: SERIAL2, symbol Connector_Generic:Conn_01x04
- added J5: CAN, symbol Connector_Generic:Conn_01x04
- added J6: PROG ESP32, symbol Connector_Generic:Conn_01x04
Connections:
- net LCD_MOSI: no longer U7.36 (IO23)
- net SCL: no longer U7.39 (IO22)
- net SDA: no longer U7.38 (IO19)
Other:
- note added: "GPS"
Changed lines of the file:
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@@
     (stroke (width 0) (type default))
   )
-  (wire (pts (xy 361.188 93.726) (xy 364.998 93.726))
+  (wire (pts (xy 171.958 71.12) (xy 175.768 71.12))
     (stroke (width 0) (type default))
   )
@@
     (stroke (width 0) (type default))
   )
-  (wire (pts (xy 361.188 91.186) (xy 364.998 91.186))
+  (wire (pts (xy 171.958 68.58) (xy 175.768 68.58))
     (stroke (width 0) (type default))
   )
@@
     (stroke (width 0) (type default))
   )
-  (wire (pts (xy 361.188 86.106) (xy 364.998 86.106))
+  (wire (pts (xy 171.958 63.5) (xy 175.768 63.5))
     (stroke (width 0) (type default))
   )
@@
     (stroke (width 0) (type default))
   )
+  (rectangle (start 180.848 202.184) (end 226.314 228.092)
+    (stroke (width 0) (type default))
+    (fill (type none))
+  )
   (text "Accelerometer" (at 290.83 182.372 0)
     (effects (font (size 1.27 1.27) (thickness 0.254) bold) (justify left bottom))
@@
   (text "ESP32" (at 271.018 31.496 0)
     (effects (font (size 1.27 1.27) (thickness 0.254) bold) (justify left bottom))
+  )
+  (text "GPS" (at 198.12 218.694 0)
+    (effects (font (size 3 3)) (justify left bottom))
   )
   (text "Boot Mode Configuration:\nPin        Default     Boot   Download\nGPIO0        1         1       0\nU0TXD        1         1       x\nGPIO2        0         x       0\nGPIO4        0         x       x\nMTDO         1         x       x\nGPIO5        1         1       x\nIf U0TXD, GPIO2, GPIO5 are floating, \nGPIO0 determines boot mode"
@@
     )
   )
-  (global_label "LCD_MOSI" (shape input) (at 364.998 93.726 0) (fields_autoplaced)
+  (global_label "LCD_MOSI" (shape input) (at 175.768 71.12 0) (fields_autoplaced)
     (effects (font (size 1.27 1.27)) (justify left))
-    (property "Intersheetrefs" "${INTERSHEET_REFS}" (at 376.543 93.6466 0)
+    (property "Intersheetrefs" "${INTERSHEET_REFS}" (at 187.313 71.0406 0)
       (effects (font (size 1.27 1.27)) (justify left) hide)
     )
@@
     )
   )
-  (global_label "SCL" (shape input) (at 364.998 91.186 0) (fields_autoplaced)
+  (global_label "SCL" (shape input) (at 175.768 68.58 0) (fields_autoplaced)
     (effects (font (size 1.27 1.27)) (justify left))
-    (property "Intersheetrefs" "${INTERSHEET_REFS}" (at 370.9187 91.1066 0)
+    (property "Intersheetrefs" "${INTERSHEET_REFS}" (at 181.6887 68.5006 0)
       (effects (font (size 1.27 1.27)) (justify left) hide)
     )
@@
     )
   )
-  (global_label "SDA" (shape input) (at 364.998 86.106 0) (fields_autoplaced)
+  (global_label "SDA" (shape input) (at 175.768 63.5 0) (fields_autoplaced)
     (effects (font (size 1.27 1.27)) (justify left))
-    (property "Intersheetrefs" "${INTERSHEET_REFS}" (at 370.9792 86.0266 0)
+    (property "Intersheetrefs" "${INTERSHEET_REFS}" (at 181.7492 63.4206 0)
       (effects (font (size 1.27 1.27)) (justify left) hide)
     )
@@
         (path "/8920b97c-b80b-47c5-aaa4-fe68c48cd11a"
           (reference "#PWR020") (unit 1)
+        )
+      )
+    )
+  )
+  (symbol (lib_id "Connector_Generic:Conn_01x04") (at 60.96 83.566 0) (unit 1)
+    (in_bom yes) (on_board yes) (dnp no) (fields_autoplaced)
+    (property "Reference" "J3" (at 62.992 84.201 0)
+      (effects (font (size 1.27 1.27)) (justify left))
+    )
+    (property "Value" "SERIAL1" (at 62.992 86.741 0)
+      (effects (font (size 1.27 1.27)) (justify left))
+    )
+    (property "Footprint" "" (at 60.96 83.566 0)
+      (effects (font (size 1.27 1.27)) hide)
+    )
+    (property "Datasheet" "~" (at 60.96 83.566 0)
+      (effects (font (size 1.27 1.27)) hide)
+    )
+    (pin "1")
+    (pin "2")
+    (pin "3")
+    (pin "4")
+    (instances
+      (project "data_logger"
+        (path "/8920b97c-b80b-47c5-aaa4-fe68c48cd11a"
+          (reference "J3") (unit 1)
         )
       )
@@
     )
   )
+  (symbol (lib_id "Connector_Generic:Conn_01x04") (at 61.214 52.324 0) (unit 1)
+    (in_bom yes) (on_board yes) (dnp no) (fields_autoplaced)
+    (property "Reference" "J6" (at 63.246 52.959 0)
+      (effects (font (size 1.27 1.27)) (justify left))
+    )
+    (property "Value" "PROG ESP32" (at 63.246 55.499 0)
+      (effects (font (size 1.27 1.27)) (justify left))
+    )
+    (property "Footprint" "" (at 61.214 52.324 0)
+      (effects (font (size 1.27 1.27)) hide)
+    )
+    (property "Datasheet" "~" (at 61.214 52.324 0)
+      (effects (font (size 1.27 1.27)) hide)
+    )
+    (pin "1")
+    (pin "2")
+    (pin "3")
+    (pin "4")
+    (instances
+      (project "data_logger"
+        (path "/8920b97c-b80b-47c5-aaa4-fe68c48cd11a"
+          (reference "J6") (unit 1)
+        )
+      )
+    )
+  )
   (symbol (lib_id "power:GND") (at 297.688 59.436 0) (unit 1)
     (in_bom yes) (on_board yes) (dnp no)
@@
         (path "/8920b97c-b80b-47c5-aaa4-fe68c48cd11a"
           (reference "#PWR014") (unit 1)
+        )
+      )
+    )
+  )
+  (symbol (lib_id "Connector_Generic:Conn_01x04") (at 60.452 110.49 0) (unit 1)
+    (in_bom yes) (on_board yes) (dnp no) (fields_autoplaced)
+    (property "Reference" "J5" (at 62.484 111.125 0)
+      (effects (font (size 1.27 1.27)) (justify left))
+    )
+    (property "Value" "CAN" (at 62.484 113.665 0)
+      (effects (font (size 1.27 1.27)) (justify left))
+    )
+    (property "Footprint" "" (at 60.452 110.49 0)
+      (effects (font (size 1.27 1.27)) hide)
+    )
+    (property "Datasheet" "~" (at 60.452 110.49 0)
+      (effects (font (size 1.27 1.27)) hide)
+    )
+    (pin "1")
+    (pin "2")
+    (pin "3")
+    (pin "4")
+    (instances
+      (project "data_logger"
+        (path "/8920b97c-b80b-47c5-aaa4-fe68c48cd11a"
+          (reference "J5") (unit 1)
         )
       )
@@
     )
   )
+  (symbol (lib_id "Connector_Generic:Conn_01x04") (at 61.722 96.266 0) (unit 1)
+    (in_bom yes) (on_board yes) (dnp no) (fields_autoplaced)
+    (property "Reference" "J4" (at 64.77 96.901 0)
+      (effects (font (size 1.27 1.27)) (justify left))
+    )
+    (property "Value" "SERIAL2" (at 64.77 99.441 0)
+      (effects (font (size 1.27 1.27)) (justify left))
+    )
+    (property "Footprint" "" (at 61.722 96.266 0)
+      (effects (font (size 1.27 1.27)) hide)
+    )
+    (property "Datasheet" "~" (at 61.722 96.266 0)
+      (effects (font (size 1.27 1.27)) hide)
+    )
+    (pin "1")
+    (pin "2")
+    (pin "3")
+    (pin "4")
+    (instances
+      (project "data_logger"
+        (path "/8920b97c-b80b-47c5-aaa4-fe68c48cd11a"
+          (reference "J4") (unit 1)
+        )
+      )
+    )
+  )
   (symbol (lib_id "power:GND") (at 305.308 88.646 0) (unit 1)
     (in_bom yes) (on_board yes) (dnp no)
@@
         )
       )
+    )
+  )
+  (symbol (lib_id "Connector_Generic:Conn_01x04") (at 60.198 69.342 0) (unit 1)
+    (in_bom yes) (on_board yes) (dnp no) (fields_autoplaced)
+    (property "Reference" "J2" (at 62.23 69.977 0)
+      (effects (font (size 1.27 1.27)) (justify left))
+    )
+    (property "Value" "I2C" (at 62.23 72.517 0)
+      (effects (font (size 1.27 1.27)) (justify left))
+    )
+    (property "Footprint" "" (at 60.198 69.342 0)
+      (effects (font (size 1.27 1.27)) hide)
+    )
+    (property "Datasheet" "~" (at 60.198 69.342 0)
+      (effects (font (size 1.27 1.27)) hide)
+    )
+    (pin "1")
+    (pin "2")
+    (pin "3")
+    (pin "4")
+    (instances
+      (project "data_logger"
+        (path "/8920b97c-b80b-47c5-aaa4-fe68c48cd11a"
+          (reference "J2") (unit 1)
+        )
+      )

Commit message: more schematic work
Parts:
- removed Q2: MBT3904DW1, Package_TO_SOT_SMD:SOT-363_SC-70-6, symbol Transistor_BJT:MBT3904DW1
- removed R13, R14, R37: 10k, Resistor_SMD:R_0603_1608Metric, symbol Device:R
- added C15: 100nF, Capacitor_SMD:C_0603_1608Metric, symbol Device:C
- added J7, J8: Conn_01x03, symbol Connector_Generic:Conn_01x03
- added R22: 10k, Resistor_SMD:R_0603_1608Metric, symbol Device:R
- added S26: TL3342F160QG, Button_Switch_SMD:SW_SPST_TL3342, symbol Switch:SW_Push
- added U6: NEO-M9N, RF_GPS:ublox_NEO, symbol RF_GPS:NEO-M9N
- R38: value 2k2 -> 20k
Connections:
- net +3.3V: now also J6.4 (Pin_4), R22.2
- net GND: now also J6.1 (Pin_1), C15.1, S26.1
- net IO0: now also C15.2, R22.1, S26.2
- net ESP_TX_OUT: now reaches J6.2 (Pin_2)
- net ESP_TX_OUT: now also J7.1 (Pin_1)
- net ESP_RX_OUT: now reaches J6.3 (Pin_3)
- net ESP_RX_OUT: now also J8.1 (Pin_1)
- net ADC_BAT: no longer names the net of U7.5 (SENSOR_VP)
- net LCD_BL: no longer names the net of U7.24 (IO4)
- net LCD_CS: no longer names the net of U7.34 (IO5)
- net LCD_DC: no longer names the net of U7.28 (SD2/IO9)
- net LCD_EN: no longer names the net of U7.29 (SD3/IO10)
- net SW_5: no longer names the net of U7.18 (IO12)
- net SW_A: no longer names the net of U7.6 (SENSOR_CAPP)
- net SW_B: no longer names the net of U7.7 (SENSOR_CAPN)
- net SW_C: no longer names the net of U7.8 (SENSOR_VN)
- net USB_RXD renamed U0RXD
- net U0RXD: now also J8.2 (Pin_2)
- net USB_TXD renamed U0TXD
- net U0TXD: now also J7.2 (Pin_2)
- new net: U6.10 (GND), U6.12 (GND), U6.13 (GND), U6.24 (GND)
- new net ESP_RX: J8.3 (Pin_3)
- new net ESP_TX: J7.3 (Pin_3)
Other:
- note added: "With great thanks to: https://github.com/CoretechR/OMOTE.git https://github.com/averywallis/Feather-NEO-M9N-GPS.git"
- note removed: "With great thanks to: https://github.com/CoretechR/OMOTE.git"
- moved on the sheet: C13, C14, C21, C22, J2, J6, LS1, U2

Commit message: more layout
Parts:
- removed U6: NEO-M9N, RF_GPS:ublox_NEO, symbol RF_GPS:NEO-M9N
- added ANT1: U.FL, UFLRSMT10, symbol Feather-NEO-M9N-GPS-rescue:U.FL-SamacSys_Parts
- added BT1: Battery_Cell, Battery:BatteryHolder_Seiko_MS621F, symbol Device:Battery_Cell
- added C1, C2: 1uF, Capacitor_SMD:C_0603_1608Metric, symbol Device:C
- added C3: 47pF, Capacitor_SMD:C_0603_1608Metric, symbol Device:C
- added D1: D_Schottky, Diode_SMD:D_SOD-323F, symbol Device:D_Schottky
- added D5: BAT60AE6327HTSA1, SOD2513X110N, symbol Device:D_Schottky
- added L1: 27nH, Inductor_SMD:L_0805_2012Metric, symbol Feather-NEO-M9N-GPS-rescue:INDUCTOR-pspice
- added R1, R16, R17, R18, R19, R2, R3, R4: 33, Resistor_SMD:R_0402_1005Metric, symbol Device:R_US
- added R14: 10k, Resistor_SMD:R_0603_1608Metric, symbol Device:R_US
- added R3 (x2): 10k, Resistor_SMD:R_0805_2012Metric, symbol Device:R
- added R7: 10, Resistor_SMD:R_0603_1608Metric, symbol Device:R_US
- added R9: 1k, Resistor_SMD:R_0603_1608Metric, symbol Device:R_US
- added U1: NEO-M9N, Feather-NEO-M9N-GPS:NEO-M9N, symbol Feather-NEO-M9N-GPS-rescue:u-blox_NEO-M9N-RF_GPS
Connections:
- net +3.3V: now also R3.1, R3.1
- net +5V: now also C3.2, U2.1 (VIN), U2.3 (CE)
- net GND: now also ANT1.1, ANT1.2, BT1.2 (-), C1.1, C2.1, C3.1, U1.10 (GND), U1.12 (GND), U1.13 (GND), U1.24 (GND)
- net SCL: now also R2.1, R3.2
- net SDA: now also R1.1, R3.2
- new net: R1.2, U1.18 (SDA/~{SPI_CS})
- new net: R18.2, U1.3 (TIMEPULSE)
- new net: R14.1, U1.2 (D_SEL)
- new net: R17.2, U1.4 (EXTINT)
- new net: R2.2, U1.19 (SCL/SPI_CLK)
- new net: R4.2, U1.20 (TXD/SPI_MISO)
- new net: D1.1 (K), R9.2
- new net: R16.2, U1.8 (~{RESET})
- new net: C3.2, L1.2, R7.2
- new net: R7.1, U1.9 (VCC_RF)
- new net: R3.2, U1.21 (RXD/SPI_MOSI)
- new net: R19.2, U1.1 (~{SAFEBOOT})
- new net +3.2V: R14.2
- new net +3V3: C1.2, D1.2 (A), D5.1 (K), U1.23 (VCC)
- new net BACKUP: BT1.1 (+), C2.2, R9.1
- new net Backup: U1.22 (V_BCKP)
- new net INT: R17.1
- new net PPS: R18.1
- new net RF: ANT1.3, L1.1, U1.11 (RF_IN)
- new net RX: R4.1
- new net TX: R3.1
- new net ~{RESET_GPS}: R16.1
- new net ~{SAFE}: R19.1
- no-connect marks 14 -> 18
Other:
- note added: "CAN BUS"
- note added: "Diode prevents reverse powering Feather"
- note added: "NEO-M9N-GPS"
- note added: "With thanks to: https://github.com/CoretechR/OMOTE.git https://github.com/averywallis/Feather-NEO-M9N-GPS.git"
- note removed: "GPS"
- note removed: "With great thanks to: https://github.com/CoretechR/OMOTE.git https://github.com/averywallis/Feather-NEO-M9N-GPS.git"
- moved on the sheet: AE1, C10, C13, C14, C15, C17, C18, C19, C21, C22, C3, C6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

Commit message: finishing pcb layout
Parts:
- removed AE1: Antenna, mkern:RFANT5220110A2T, symbol Device:Antenna
- removed C14: 100nF, Capacitor_SMD:C_0603_1608Metric, symbol Device:C
- removed C18, C19: 1.2pF, Capacitor_SMD:C_0603_1608Metric, symbol Device:C
- removed C21, C3: 10uF, Capacitor_SMD:C_0805_2012Metric, symbol Device:C
- removed D3: LED, LED_SMD:LED_0603_1608Metric, symbol Device:LED
- removed D5: BAT60AE6327HTSA1, SOD2513X110N, symbol Device:D_Schottky
- removed J2: I2C, symbol Connector_Generic:Conn_01x04
- removed J4: SERIAL2, symbol Connector_Generic:Conn_01x04
- removed J6: PROG ESP32, symbol Connector_Generic:Conn_01x04
- removed R1, R16, R17, R18, R19, R2, R3, R4: 33, Resistor_SMD:R_0402_1005Metric, symbol Device:R_US
- removed R36: 0, Resistor_SMD:R_0603_1608Metric, symbol Device:R
- removed R38: 20k, Resistor_SMD:R_0603_1608Metric, symbol Device:R
- removed U1: Teensy4.1, teensy:Teensy41, symbol teensy:Teensy4.1
- removed U2: XC6220B331, Package_TO_SOT_SMD:SOT-23-5, symbol Regulator_Linear:XC6220B331MR
- removed U7: ESP32-PICO-D4, mkern:QFN-48-1EP_7x7mm_P0.5mm_EP5.3x5.3mm_ThermalVias_MR, symbol RF_Module:ESP32-PICO-D4
- added C10: 100nF, Capacitor_SMD:C_0603_1608Metric, symbol Device:C
- added D3: LED BLU, LED_SMD:LED_0603_1608Metric, symbol Device:LED
- added D3: LED GRN, LED_SMD:LED_0603_1608Metric, symbol Device:LED
- added D3: LED RED, LED_SMD:LED_0603_1608Metric, symbol Device:LED
- added J6: SD_Card, Connector_Card:TF-SMD_TF-013-A, symbol Connector:SD_Card
- added JP1, JP2: SolderJumper_3_Open, Jumper:SolderJumper-3_P1.3mm_Open_Pad1.0x1.5mm, symbol Jumper:SolderJumper_3_Open
- added R38 (x4): 20k, Resistor_SMD:R_0603_1608Metric, symbol Device:R
- added U4: LD1117S18TR_SOT223, Package_TO_SOT_SMD:SOT-223-3_TabPin2, symbol Regulator_Linear:LD1117S18TR_SOT223
- added U6: DEV-15583, MODULE_DEV-15583, symbol DEV-15583:DEV-15583
- added U7: ESP32-WROOM-32D, RF_Module:ESP32-WROOM-32D, symbol RF_Module:ESP32-WROOM-32D
- ANT1: MPN U.FL-R-SMT(10) -> (none)
- BT1: MPN MS621FE-FL11E -> (none); now left out of the parts list
- C1, C2: LCSC (none) -> C15849; MPN CL10A105KA8NNNC -> (none)
- C10, C15, C17, C22: LCSC (none) -> C14663
- C13, C6: LCSC (none) -> C15850
- C3: LCSC (none) -> C1671; MPN GRM1885C1H470FA01J -> (none)
- D1: footprint Diode_SMD:D_SOD-323F -> Diode_SMD:D_SOD-123; LCSC (none) -> C8598; MPN PMEG4005EJF -> (none)
- J1: renamed from J3; footprint (none) -> Connector_PinHeader_2.54mm:PinHeader_1x04_P2.54mm_Vertical; now left out of the parts list
- J2: footprint 4pin:my_4_tab_edge -> Connector_PinHeader_2.54mm:PinHeader_1x04_P2.54mm_Vertical
- J3: renamed from J8; footprint (none) -> Connector_PinHeader_2.54mm:PinHeader_1x03_P2.54mm_Vertical
- J4: renamed from J7; footprint (none) -> Connector_PinHeader_2.54mm:PinHeader_1x03_P2.54mm_Vertical
- J5: value CAN -> PROG ESP32; footprint (none) -> Connector_PinHeader_2.54mm:PinHeader_1x04_P2.54mm_Vertical
- L1: LCSC (none) -> C1330812; MPN CE201210-27NJ -> (none)
- LS1: footprint (none) -> Buzzer_Beeper:BUZ-SMD_5P-L15.0-W15.0-P13.7-BL; LCSC (none) -> C482341
- R14: LCSC (none) -> C25804; MPN ESR03EZPJ103 -> (none)
- R22: LCSC (none) -> C25804
- R3, R7: footprint Resistor_SMD:R_0805_2012Metric -> Resistor_SMD:R_0603_1608Metric
- R7: LCSC (none) -> C22859; MPN ESR03EZPF10R0 -> (none)
- R9: LCSC (none) -> C21190; MPN ESR03EZPJ102 -> (none)
- S26: footprint Button_Switch_SMD:SW_SPST_TL3342 -> Button_Switch_SMD:SW_SPST_B3SL-1022P; LCSC (none) -> C318884
- U5: footprint XDCR_LIS3DHTR -> LIS3DHTR:LGA-16_L3.0-W3.0-P0.50-TL; LCSC (none) -> C15134; MAXIMUM_PACKAGE_HEIGHT 1mm -> (none); PARTREV 2 -> (none); STANDARD Manufacturer Recommendations -> (none)
Connections:
- net +3.2V is gone; now on net +3.3V: R14.2
- net Backup is gone; now on net BACKUP: U1.22 (V_BCKP)
- net +3.3V: now also J5.4 (Pin_4), J6.4 (VDD), JP1.3 (B), JP2.3 (B), R38.2, U4.2 (VO), U6.3.3V_2, U7.2 (VDD)
- net +5V: now also C10.1, JP1.1 (A), JP2.1 (A), U4.3 (VI), U6.VIN; no longer J2.4 (Pin_4)
- net ACC_INT: now also U6.8
- net CAN_RX: now also U6.0
- net CAN_TX: now also U6.1
- net ESP_EN: now also U7.3 (EN)
- net ESP_RX: now also U6.15
- net ESP_RX_OUT: now also J5.3 (Pin_3)
- net ESP_TX: now also U6.14
- net ESP_TX_OUT: now also J5.2 (Pin_2)
- net GND: now also J1.4 (Pin_4), J5.1 (Pin_1), LS1.1, C10.2, J6.3 (VSS), J6.6 (VSS), R38.1, R38.1, R38.1, U4.1 (GND), U6.G1, U6.G3, U7.1 (GND), U7.15 (GND), U7.38 (GND), U7.39 (GND)
- net IO0: now also U7.25 (IO0)
- net PPS: now also U1.3 (TIMEPULSE), U6.20
- net SCL: now also U1.19 (SCL/SPI_CLK), U6.19
- net SDA: now also U1.18 (SDA/~{SPI_CS}), U6.18
- net U0RXD: now also U7.34 (RXD0/IO3)
- net U0TXD: now also U7.35 (TXD0/IO1)
- net EXTINT: now reaches U1.4 (EXTINT)
- net EXTINT: now also U6.22
- net RESET_GPS: now reaches U1.8 (~{RESET})
- net RESET_GPS: now also U6.23
- net SPK: now reaches LS1.2
- net SPK: now also U6.9
- net at J1.1 (Pin_1): now also JP1.2 (C)
- net RX1: now reaches J1.2 (Pin_2)
- net TX1: now reaches J1.3 (Pin_3)
- new net: D3.1 (K), R38.2 (x3)
- new net: D3.2 (A), U7.24 (IO2)
- new net: J2.4 (Pin_4), JP2.2 (C)
- new net CLK: J6.5 (CLK), U6.13
- new net CS: J6.1 (CD/DAT3), U6.10
- new net LED1: D3.2 (A), U6.17
- new net LED2: D3.2 (A), U6.16
- new net MISO: J6.7 (DAT0), R38.1, U6.12
- new net MOSI: J6.2 (CMD), U6.11
- no-connect marks 18 -> 44
Other:
- note added: "MP2 SER"
- note removed: "Diode prevents reverse powering Feather"
- moved on the sheet: ANT1, BT1, C1, C10, C13, C15, C17, C2, C22, C3, C6, D1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

Commit message: finalized pcb
Parts:
- removed C10: 100nF, Capacitor_SMD:C_0603_1608Metric, symbol Device:C
- added C10: C_Polarized_Small_US, Capacitor_Tantalum_SMD:CP_EIA-3216-18_Kemet-A, symbol Device:C_Polarized_Small_US
- ANT1: footprint UFLRSMT10 -> RF_Antenna:molex_ 0732519780
- U4: LCSC C80598 -> C2984862
Connections:
- net +3V3 is gone; now on net +3.3V: C1.2, D1.2 (A), U1.23 (VCC)
- net +3.3V: now also C10.1; no longer C6.1
- net +5V: now also C6.1
- net GND: now also C10.2
Other:
- note added: "Disconnect RX/TX lines for serial program"
- moved on the sheet: C13, C15, C22, J1, J3, J4, JP1, LS1, R22, R38, S26, U4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

Commit message: finished design
Connections:
- net ESP_RX: now also U6.14; no longer U6.15
- net ESP_TX: now also U6.15; no longer U6.14
Other:
- moved on the sheet: C10, C17, C6, R38, U4, U5, U6

Commit message: manufacturing files
Parts:
- J6: LCSC (none) -> C961683
- U6: now left out of the parts list
- U7: LCSC (none) -> C529578
Changed lines of the file:
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@@
+      (effects (font (size 1.27 1.27)) hide)
+    )
+    (property "LCSC" "C529578" (at 287.401 82.677 0)
       (effects (font (size 1.27 1.27)) hide)
     )
@@
   )
   (symbol (lib_id "DEV-15583:DEV-15583") (at 84.709 65.786 0) (unit 1)
-    (in_bom yes) (on_board yes) (dnp no) (fields_autoplaced)
+    (in_bom no) (on_board yes) (dnp no) (fields_autoplaced)
     (property "Reference" "U6" (at 84.709 41.656 0)
       (effects (font (size 1.27 1.27)))
@@
       (effects (font (size 1.27 1.27)) hide)
     )
+    (property "LCSC" "C961683" (at 102.489 110.617 0)
+      (effects (font (size 1.27 1.27)) hide)
+    )

Commit message: manufacturing files
Parts:
- J3, J4, J5: now left out of the parts list
- J6: LCSC C961683 -> C444917
- R38: now in the parts list
Changed lines of the file:
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@@
   )
   (symbol (lib_id "Device:R") (at 24.765 111.125 180) (unit 1)
-    (in_bom no) (on_board yes) (dnp no) (fields_autoplaced)
+    (in_bom yes) (on_board yes) (dnp no) (fields_autoplaced)
     (property "Reference" "R38" (at 26.543 110.49 0)
       (effects (font (size 1.27 1.27)) (justify right))
@@
   )
   (symbol (lib_id "Connector_Generic:Conn_01x04") (at 250.444 147.955 180) (unit 1)
-    (in_bom yes) (on_board yes) (dnp no) (fields_autoplaced)
+    (in_bom no) (on_board yes) (dnp no) (fields_autoplaced)
     (property "Reference" "J5" (at 250.444 137.541 0)
       (effects (font (size 1.27 1.27)) hide)
@@
   )
   (symbol (lib_id "Device:R") (at 320.421 63.627 0) (mirror x) (unit 1)
-    (in_bom no) (on_board yes) (dnp no) (fields_autoplaced)
+    (in_bom yes) (on_board yes) (dnp no) (fields_autoplaced)
     (property "Reference" "R38" (at 318.643 62.992 0)
       (effects (font (size 1.27 1.27)) (justify right))
@@
       (effects (font (size 1.27 1.27)) hide)
     )
-    (property "LCSC" "C961683" (at 102.489 110.617 0)
+    (property "LCSC" "C444917" (at 102.489 110.617 0)
       (effects (font (size 1.27 1.27)) hide)
     )
@@
   )
   (symbol (lib_id "Device:R") (at 42.545 111.125 180) (unit 1)
-    (in_bom no) (on_board yes) (dnp no) (fields_autoplaced)
+    (in_bom yes) (on_board yes) (dnp no) (fields_autoplaced)
     (property "Reference" "R38" (at 44.323 110.49 0)
       (effects (font (size 1.27 1.27)) (justify right))
@@
   )
   (symbol (lib_id "Device:R") (at 73.66 118.237 270) (unit 1)
-    (in_bom no) (on_board yes) (dnp no)
+    (in_bom yes) (on_board yes) (dnp no)
     (property "Reference" "R38" (at 74.93 120.777 90)
       (effects (font (size 1.27 1.27)) (justify right))
@@
   )
   (symbol (lib_id "Connector_Generic:Conn_01x03") (at 221.361 137.287 180) (unit 1)
-    (in_bom yes) (on_board yes) (dnp no) (fields_autoplaced)
+    (in_bom no) (on_board yes) (dnp no) (fields_autoplaced)
     (property "Reference" "J3" (at 221.361 132.715 0)
       (effects (font (size 1.27 1.27)))
@@
   )
   (symbol (lib_id "Connector_Generic:Conn_01x03") (at 221.361 147.447 180) (unit 1)
-    (in_bom yes) (on_board yes) (dnp no) (fields_autoplaced)
+    (in_bom no) (on_board yes) (dnp no) (fields_autoplaced)
     (property "Reference" "J4" (at 221.361 142.875 0)
       (effects (font (size 1.27 1.27)))
