File: data_logger.kicad_sch (KiCad schematic)
At the start: 48 parts, among them J1 SERIAL1, J2 Conn_01x04, J3 Conn_01x03, J4 Conn_01x03, J5 PROG ESP32, J6 SD_Card, U1 NEO-M9N, U2 TJA1050T/CM,118, U4 LD1117S18TR_SOT223, U5 LIS3DHTR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

Commit message: ORDERED FROM JLCPCB
Parts:
- ANT1, U1: now left out of the parts list
Changed lines of the file:
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@@
   )
   (symbol (lib_id "Feather-NEO-M9N-GPS-rescue:U.FL-SamacSys_Parts") (at 51.435 173.355 0) (unit 1)
-    (in_bom yes) (on_board yes) (dnp no)
+    (in_bom no) (on_board yes) (dnp no)
     (property "Reference" "ANT1" (at 60.325 144.145 0)
       (effects (font (size 1.27 1.27)))
@@
   )
   (symbol (lib_id "Feather-NEO-M9N-GPS-rescue:u-blox_NEO-M9N-RF_GPS") (at 109.855 159.385 0) (unit 1)
-    (in_bom yes) (on_board yes) (dnp no)
+    (in_bom no) (on_board yes) (dnp no)
     (property "Reference" "U1" (at 108.585 135.255 0)
       (effects (font (size 1.27 1.27)))
