File: data_logger.kicad_pcb (KiCad board)
At the start: 2 copper layers, 1 part, among them U1 Teensy4.1

Commit message: finishing pcb layout
Parts:
- added ANT1: U.FL, Feather-NEO-M9N-GPS:UFLRSMT10, F.Cu at (89.7, 95.0)
- added BT1: Battery_Cell, Battery:BatteryHolder_Seiko_MS621F, F.Cu at (120.7, 82.5)
- added C1: 1uF, Capacitor_SMD:C_0603_1608Metric, F.Cu at (115.7, 87.0)
- added C12: 100nF, Capacitor_SMD:C_0603_1608Metric, F.Cu at (156.7, 127.8)
- added C13: 100nF, Capacitor_SMD:C_0603_1608Metric, F.Cu at (148.4, 127.8)
- added C14: 100nF, Capacitor_SMD:C_0603_1608Metric, F.Cu at (95.6, 127.9)
- added C2: 47pF, Capacitor_SMD:C_0603_1608Metric, F.Cu at (97.3, 88.2)
- added C3: 1uF, Capacitor_SMD:C_0603_1608Metric, F.Cu at (113.9, 81.1)
- added C5: 10uF, Capacitor_SMD:C_0805_2012Metric, F.Cu at (92.5, 121.5)
- added C6: 100nF, Capacitor_SMD:C_0603_1608Metric, F.Cu at (118.2, 118.6)
- added C7: 100nF, Capacitor_SMD:C_0603_1608Metric, F.Cu at (156.9, 76.4)
- added C8: 10uF, Capacitor_SMD:C_0805_2012Metric, F.Cu at (153.5, 76.1)
- added C9: 100nF, Capacitor_SMD:C_0603_1608Metric, F.Cu at (118.2, 121.5)
- added D1: LED RED, LED_SMD:LED_0603_1608Metric, F.Cu at (120.7, 94.3)
- added D2: D_Schottky, Diode_SMD:D_SOD-123, F.Cu at (116.2, 82.7)
- added D3: LED GRN, LED_SMD:LED_0603_1608Metric, F.Cu at (122.9, 94.4)
- added D4: LED BLU, LED_SMD:LED_0603_1608Metric, F.Cu at (137.3, 91.6)
- added D5: LED BLU, LED_SMD:LED_0603_1608Metric, F.Cu at (135.5, 95.9)
- added J1: SERIAL1, Connector_PinHeader_2.54mm:PinHeader_1x04_P2.54mm_Vertical, F.Cu at (121.1, 130.2)
- added J2: Conn_01x04, Connector_PinHeader_2.54mm:PinHeader_1x04_P2.54mm_Vertical, F.Cu at (101.1, 130.1)
- added J3: Conn_01x03, Connector_PinHeader_2.54mm:PinHeader_1x03_P2.54mm_Vertical, F.Cu at (131.6, 88.3)
- added J4: Conn_01x03, Connector_PinHeader_2.54mm:PinHeader_1x03_P2.54mm_Vertical, F.Cu at (131.6, 77.9)
- added J5: PROG ESP32, Connector_PinHeader_2.54mm:PinHeader_1x04_P2.54mm_Vertical, F.Cu at (126.5, 81.5)
- added J6: SD_Card, Connector_Card:TF-SMD_TF-013-A, F.Cu at (149.2, 106.9)
- added JP1: SolderJumper_3_Open, Jumper:SolderJumper-3_P1.3mm_Open_Pad1.0x1.5mm, F.Cu at (118.2, 126.0)
- added JP2: SolderJumper_3_Open, Jumper:SolderJumper-3_P1.3mm_Open_Pad1.0x1.5mm, F.Cu at (114.2, 125.9)
- added L1: 27nH, Inductor_SMD:L_0805_2012Metric, F.Cu at (97.3, 95.0)
- added LS1: Speaker, Buzzer_Beeper:BUZ-SMD_5P-L15.0-W15.0-P13.7-BL, F.Cu at (132.9, 123.9)
- added R1: 20k, Resistor_SMD:R_0603_1608Metric, F.Cu at (118.6, 94.2)
- added R10: 10k, Resistor_SMD:R_0603_1608Metric, F.Cu at (154.9, 127.8)
- added R11: 10k, Resistor_SMD:R_0603_1608Metric, F.Cu at (146.1, 127.8)
- added R12: 20k, Resistor_SMD:R_0603_1608Metric, F.Cu at (135.4, 94.2)
- added R13: 20k, Resistor_SMD:R_0603_1608Metric, F.Cu at (135.6, 91.6)
- added R13: 20k, Resistor_SMD:R_0603_1608Metric, F.Cu at (133.8, 113.2)
- added R2: 10k, Resistor_SMD:R_0603_1608Metric, F.Cu at (110.0, 124.9)
- added R3: 1k, Resistor_SMD:R_0603_1608Metric, F.Cu at (114.0, 84.4)
- added R4: 20k, Resistor_SMD:R_0603_1608Metric, F.Cu at (125.0, 94.4)
- added R5: 120, Resistor_SMD:R_0603_1608Metric, F.Cu at (104.6, 127.4)
- added R6: 10, Resistor_SMD:R_0603_1608Metric, F.Cu at (97.3, 91.4)
- added R7: 10k, Resistor_SMD:R_0603_1608Metric, F.Cu at (97.2, 83.0)
- added R8: 10k, Resistor_SMD:R_0603_1608Metric, F.Cu at (112.8, 116.7)
- added R9: 10k, Resistor_SMD:R_0603_1608Metric, F.Cu at (116.8, 116.3)
- added S1: TL3342F160QG, Button_Switch_SMD:SW_SPST_B3SL-1022P, F.Cu at (154.5, 121.5)
- added S2: TL3342F160QG, Button_Switch_SMD:SW_SPST_B3SL-1022P, F.Cu at (146.5, 121.4)
- added U3: NEO-M9N, Feather-NEO-M9N-GPS:NEO-M9N, F.Cu at (105.7, 88.1)
- added U4: LD1117S18TR_SOT223, Package_TO_SOT_SMD:SOT-223-3_TabPin2, F.Cu at (98.7, 123.0)
- added U5: LIS3DHTR, LIS3DHTR:LGA-16_L3.0-W3.0-P0.50-TL, F.Cu at (115.4, 120.1)
- added U6: DEV-15583, DEV-15583:MODULE_DEV-15583, F.Cu at (113.0, 106.3)
- added U7: ESP32-WROOM-32D, RF_Module:ESP32-WROOM-32D, F.Cu at (149.2, 87.0)
- U1: value Teensy4.1 -> TJA1050T/CM,118; footprint teensy:Teensy41 -> Package_SO:SOIC-8_3.9x4.9mm_P1.27mm
- moved U1 32.3 mm to (106.8, 120.3), turned to -90 degrees
Connections:
- U1 pad 1: unconnected-(U1-GND-Pad1) -> CAN_TX
- U1 pad 2: unconnected-(U1-0_RX1_CRX2_CS1-Pad2) -> GND
- U1 pad 3: unconnected-(U1-1_TX1_CTX2_MISO1-Pad3) -> +3.3V
- U1 pad 4: unconnected-(U1-2_OUT2-Pad4) -> CAN_RX
- U1 pad 6: unconnected-(U1-4_BCLK2-Pad6) -> CAN_LO
- U1 pad 7: unconnected-(U1-5_IN2-Pad7) -> CAN_HI
- U1 pad 8: unconnected-(U1-6_OUT1D-Pad8) -> Net-(U1-Rs)
Routing:
- net GND: track 0.00 -> 64.4 mm, vias 0 -> 29
- net +5V: track 0.00 -> 58.6 mm, vias 0 -> 2
- net ESP_EN: track 0.00 -> 54.8 mm
- net IO0: track 0.00 -> 38.8 mm
- net SCL: track 0.00 -> 36.7 mm, vias 0 -> 1
- net SDA: track 0.00 -> 35.7 mm, vias 0 -> 1
- net U0TXD: track 0.00 -> 29.5 mm, vias 0 -> 1
- net U0RXD: track 0.00 -> 26.6 mm, vias 0 -> 1
- net PPS: track 0.00 -> 23.4 mm
- net CLK: track 0.00 -> 22.8 mm, vias 0 -> 1
- net CS: track 0.00 -> 21.3 mm
- net EXTINT: track 0.00 -> 19.7 mm
- net ESP_TX: track 0.00 -> 19.1 mm
- net MOSI: track 0.00 -> 18.3 mm
- net +3.3V: track 0.00 -> 15.7 mm
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- added copper zone on F.Cu, net +3.3V
- added copper zone on B.Cu, net GND
Other:
- rule pad_to_mask_clearance: 0 -> 0.051

Commit message: finalized pcb
Parts:
- removed C14: 100nF, Capacitor_SMD:C_0603_1608Metric
- removed C5: 10uF, Capacitor_SMD:C_0805_2012Metric
- added C10: C_Polarized_Small_US, Capacitor_Tantalum_SMD:CP_EIA-3216-18_Kemet-A, F.Cu at (85.1, 121.7)
- added C4: 10uF, Capacitor_SMD:C_0805_2012Metric, F.Cu at (87.9, 129.0)
- added REF**: MountingHole_3.2mm_M3, MountingHole:MountingHole_3.2mm_M3, F.Cu at (155.4, 128.0)
- added REF**: MountingHole_3.2mm_M3, MountingHole:MountingHole_3.2mm_M3, F.Cu at (82.8, 128.5)
- ANT1: footprint Feather-NEO-M9N-GPS:UFLRSMT10 -> RF_Antenna:molex_ 0732519780
- moved C6 7.48 mm to (110.8, 119.2)
- moved JP1 7.48 mm to (110.7, 126.6)
- moved JP2 7.48 mm to (106.7, 126.5)
- moved R2 7.48 mm to (102.5, 125.5)
- moved R9 7.48 mm to (109.3, 116.8)
- moved U5 7.48 mm to (107.9, 120.6)
- moved R8 7.48 mm to (105.3, 117.3)
- moved U1 7.48 mm to (99.3, 120.8)
- moved C9 7.48 mm to (110.7, 122.1)
- moved J1 7.48 mm to (113.7, 130.7)
- moved J2 7.48 mm to (93.6, 130.6)
- moved R5 7.48 mm to (97.2, 128.0)
- moved U4 7.48 mm to (91.2, 123.6)
- moved LS1 6.96 mm to (126.0, 124.5)
- moved S1 6.96 mm to (147.6, 122.0)
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Connections:
- C3 pad 2: +3V3 -> +3.3V
- D2 pad 2: +3V3 -> +3.3V
- U3 pad 23: +3V3 -> +3.3V
Routing:
- net +3.3V: track 15.7 -> 30.2 mm
- net /RF: track 2.40 -> 13.4 mm
- net ACC_INT: track 9.35 -> 15.5 mm
- net Net-(D2-K): track 2.53 -> 8.61 mm
- net SDA: track 35.7 -> 40.4 mm
- net CAN_TX: track 8.99 -> 4.57 mm
- net CAN_RX: track 7.54 -> 5.09 mm
- net +3V3: track 2.40 -> 0.00 mm
- net SCL: track 36.7 -> 38.8 mm, vias 1 -> 0
- net EXTINT: track 19.7 -> 17.7 mm
- net +5V: track 58.6 -> 60.0 mm
- net ESP_EN: track 54.8 -> 56.1 mm, vias 0 -> 2
- net GND: track 64.4 -> 63.6 mm, vias 29 -> 41
- net IO0: track 38.8 -> 38.5 mm, vias 0 -> 2
- added copper zone on F.Cu, net GND
Other:
- board outline added: 81.2 x 58.2 mm
- board text added: "+3"
- board text added: "+5"
- board text added: "CAN_HI"
- board text added: "CAN_LO"
- board text added: "Data logger V1.0"
- board text added: "GND"
- board text added: "RX"
- board text added: "TX"
- board text added: "Vin"

Commit message: finished design
Parts:
- removed D4: LED BLU, LED_SMD:LED_0603_1608Metric
- removed the R13 at (135.6, 91.6)
- moved C2 85.5 mm to (36.1, 28.5)
- moved C3 85.5 mm to (52.6, 21.4)
- moved C4 85.5 mm to (26.7, 69.4)
- moved C9 85.5 mm to (49.5, 62.4)
- moved J1 85.5 mm to (52.5, 71.1)
- moved JP2 85.5 mm to (45.5, 66.9)
- moved R5 85.5 mm to (36.0, 68.3)
- moved R9 85.5 mm to (48.1, 57.2)
- moved U5 85.5 mm to (46.7, 61.0)
- moved ANT1 85.5 mm to (24.1, 34.4)
- moved BT1 85.5 mm to (59.4, 22.9)
- moved C1 85.5 mm to (54.5, 27.3)
- moved C10 85.5 mm to (23.9, 62.0)
- moved C12 85.5 mm to (88.6, 68.8)
- moved C6 85.5 mm to (49.6, 59.6)
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Connections:
- U6 pad 14: ESP_TX -> ESP_RX
- U6 pad 15: ESP_RX -> ESP_TX
Routing:
- net MISO: track 13.4 -> 24.9 mm, vias 0 -> 2
- net +3.3V: track 30.2 -> 23.2 mm
- net ESP_RX: track 9.27 -> 7.25 mm
- net CS: track 21.3 -> 23.0 mm
- net Net-(D4-K): track 1.65 -> 0.00 mm
- net MOSI: track 18.3 -> 19.6 mm
- net GND: track 63.6 -> 62.4 mm, vias 41 -> 40
- net +5V: track 60.0 -> 59.8 mm, vias 2 -> 4
- net SCL: track 38.8 -> 38.9 mm, vias 0 -> 2

Commit message: manufacturing files
Parts:
- added REF**: MountingHole_3.2mm_M3, MountingHole:MountingHole_3.2mm_M3, F.Cu at (21.0, 18.6)
- moved REF** 0.57 mm to (21.0, 68.9)
Routing:
- net +5V: track 59.8 -> 62.4 mm
Other:
- outline, holes or cut-outs redrawn
- board text added: "U1 CAN = 180 U4 LDO = 180 U7 ESP = 180"

Commit message: manufacturing files
Other:
- board text added: "U1 CAN = 180 U4 LDO = 180 U7 ESP = 180, x = 87.18"
- board text removed: "U1 CAN = 180 U4 LDO = 180 U7 ESP = 180"
Changed lines of the file:
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@@
     (property "ki_description" "Resistor")
     (property "ki_keywords" "R res resistor")
-    (attr smd exclude_from_bom)
+    (attr smd)
     (fp_text reference "R12" (at 0 -1.43) (layer "F.SilkS") hide
         (effects (font (size 1 1) (thickness 0.15)))
@@
     (effects (font (size 1 1) (thickness 0.2) bold) (justify left bottom))
   )
-  (gr_text "U1 CAN = 180\nU4 LDO = 180\nU7 ESP = 180" (at 35.18 79.34) (layer "F.SilkS")
+  (gr_text "U1 CAN = 180\nU4 LDO = 180\nU7 ESP = 180, x = 87.18" (at 35.18 79.34) (layer "F.SilkS")
     (effects (font (size 1 1) (thickness 0.15)) (justify left bottom))
   )

Commit message: ORDERED FROM JLCPCB
Other:
- board text added: "1"
- board text added: "U1 CAN = 180 U4 LDO = 180 U7 ESP = 180, x = 87.26"
- board text removed: "U1 CAN = 180 U4 LDO = 180 U7 ESP = 180, x = 87.18"
Changed lines of the file:
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@@
     (effects (font (size 1 1) (thickness 0.24) bold) (justify left bottom))
+  )
+  (gr_text "1" (at 32.512 57.15) (layer "F.SilkS")
+    (effects (font (size 1.5 1.5) (thickness 0.3) bold) (justify left bottom))
   )
   (gr_text "+5" (at 50.54 66.15) (layer "F.SilkS")
     (effects (font (size 1 1) (thickness 0.2) bold) (justify left bottom))
   )
-  (gr_text "U1 CAN = 180\nU4 LDO = 180\nU7 ESP = 180, x = 87.18" (at 35.18 79.34) (layer "F.SilkS")
+  (gr_text "U1 CAN = 180\nU4 LDO = 180\nU7 ESP = 180, x = 87.26" (at 35.18 79.34) (layer "F.SilkS")
     (effects (font (size 1 1) (thickness 0.15)) (justify left bottom))
   )
@@
       )
     )
-  )
-  (zone (net 0) (net_name "") (layer "F.Cu") (hatch none 0.5)
-    (connect_pads yes (clearance 0))
-    (min_thickness 0.25) (filled_areas_thickness no)
-    (keepout (tracks allowed) (vias allowed) (pads allowed) (copperpour not_allowed) (footprints allowed))
-    (fill (thermal_gap 0.5) (thermal_bridge_width 0.5))
-    (polygon
-      (pts
-        (xy 79.1216 25.424)
-        (xy 77.2928 25.424)
-        (xy 76.9372 24.3572)
-        (xy 75.4132 24.3826)
-        (xy 75.4132 25.8304)
-        (xy 75.8704 27.0496)
-        (xy 76.8864 27.0496)
-        (xy 77.1404 26.694)
-        (xy 79.0708 26.694)
-      )
-    )
