File: V1.1/data_logger.kicad_sch (KiCad schematic)
At the start: 52 parts, among them J1 SERIAL1, J2 Conn_01x04, J3 Conn_01x03, J4 Conn_01x03, J5 Conn_01x05, J6 GPS1, J7 Micro_SD_Card, U1 NEO-M9N, U2 LSM6DS3, U2 TJA1050T/CM,118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

Commit message: more firmware work
Other:
- moved on the sheet: D3, J1, JP1, JP2, LS1, R38, U6
