File: brainboardV1.0/VESC_brain_board.kicad_pcb (KiCad board)
At the start: 4 copper layers, 90.1 x 71 mm, 50 parts, among them J1 Conn_01x18, J12 Conn_01x03, J13 Conn_01x03, J14 SERIAL1, J15 Conn_01x03, J21 Conn_01x01, J22 Conn_01x01, J23 Conn_01x01, Q1 my_BC337, U1 TJA1050T/CM,118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

Commit message: finished V1.0
Parts:
- removed 10k_2, 10k_3: 10k, Resistor_SMD:R_0603_1608Metric
- added 1k_21: 1k, Resistor_SMD:R_0603_1608Metric, F.Cu at (76.3, 40.5)
- added 1k_22: 1k, Resistor_SMD:R_0603_1608Metric, F.Cu at (75.6, 34.4)
- added REF**: MountingHole_3.2mm_M3, MountingHole:MountingHole_3.2mm_M3, F.Cu at (43.0, 76.8)
- added REF**: MountingHole_3.2mm_M3, MountingHole:MountingHole_3.2mm_M3, F.Cu at (90.2, 65.5)
- added REF**: MountingHole_3.2mm_M3, MountingHole:MountingHole_3.2mm_M3, F.Cu at (90.2, 19.8)
- added REF**: MountingHole_3.2mm_M3, MountingHole:MountingHole_3.2mm_M3, F.Cu at (41.0, 36.2)
- 1k_1: footprint Resistor_SMD:R_0805_2012Metric -> Resistor_SMD:R_0603_1608Metric
- DC_2: footprint Capacitor_SMD:C_0805_2012Metric -> Capacitor_SMD:C_0603_1608Metric
- moved 10k_8 20.8 mm to (69.7, 63.3)
- moved DC_1 20.8 mm to (79.3, 68.3)
- moved S1 20.8 mm to (73.9, 68.4)
- moved J21 15.7 mm to (100.0, 75.9)
- moved VESC1 14.4 mm to (67.4, 80.5)
- moved VESC2 14.4 mm to (89.4, 80.7)
- moved J23 10.3 mm to (100.0, 59.8)
- moved J22 7.79 mm to (100.0, 67.4)
- moved R_120 3.29 mm to (76.4, 48.7)
- moved U1 3.29 mm to (71.7, 48.9)
- moved 10k_1 2.18 mm to (73.3, 45.4), turned to 180 degrees
- moved JP1 1.43 mm to (80.0, 60.1), turned to 0 degrees
- moved DC_6 0.52 mm to (101.5, 23.0)
- moved DC_5 0.52 mm to (98.2, 22.9)
- moved S11 0.30 mm to (99.7, 47.0)
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Connections:
- J12 pad 2: U0RXD -> Net-(J12-Pin_2)
- J13 pad 2: U0TXD -> Net-(J13-Pin_2)
- U11 pad 26: ESP_IO -> unconnected-(U11-IO4-Pad26)
- U2 pad 14: unconnected-(U2-12_MISO_MQSL-Pad14) -> VESC1_TX
- U2 pad 20: unconnected-(U2-13_SCK_CRX1_LED-Pad20) -> SPEAKER
- U2 pad 21: VSENSE -> VESC2_EN
- U2 pad 22: unconnected-(U2-15_A1_RX3_SPDIF_IN-Pad22) -> VESC2_ADC2
- U2 pad 23: unconnected-(U2-16_A2_RX4_SCL1-Pad23) -> VESC2_TX
- U2 pad 24: unconnected-(U2-17_A3_TX4_SDA1-Pad24) -> BUTTON
- U2 pad 28: unconnected-(U2-21_A7_RX5_BCLK1-Pad28) -> VSENSE
Routing:
- net +5V: track 143.2 -> 281.5 mm, vias 4 -> 6
- net VSENSE: track 5.37 -> 54.2 mm, vias 0 -> 3
- net VESC2_TX: track 0.00 -> 45.4 mm
- net VESC1_VCC: track 79.3 -> 122.4 mm, vias 3 -> 2
- net VESC2_ADC2: track 0.00 -> 42.4 mm
- net VESC1_TX: track 0.00 -> 40.4 mm
- net VESC2_EN: track 0.00 -> 37.8 mm
- net /CAN_RX: track 0.00 -> 30.6 mm
- net SPEAKER: track 0.00 -> 24.4 mm
- net /CAN_TX: track 0.00 -> 24.0 mm
- net VESC_+5V: track 153.7 -> 130.1 mm
- net BUTTON: track 12.0 -> 35.5 mm
- net +3.3V: track 7.64 -> 30.3 mm, vias 1 -> 8
- net Net-(CAN1-Pin_4): track 0.00 -> 12.4 mm
- net CAN_LO: track 0.00 -> 7.84 mm
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- added copper zone on In2.Cu, net +3.3V
- added copper zone on F.Cu, net GND
- added copper zone on In1.Cu, net GND
- removed copper zone on F.Cu, net +3.3V
Other:
- board size 90.1 x 71 mm -> 90.5 x 68.6 mm
- board text added: "+3.3V"
- board text added: "+5V"
- board text added: "1"
- board text added: "2"
- board text added: "3"
- board text added: "4"
- board text added: "5"
- board text added: "6"
- board text added: "BOOT"
- board text added: "CAN VOLT SELECT"
- board text added: "C_H"
- board text added: "C_L"
- board text added: "ENBL"
- board text added: "ESP32 PROG VOLT SELECT"
- board text added: "GND"
- board text added: "MPU6050"
- board text added: "PROG_Rx"
- board text added: "PROG_Tx"
- board text added: "Rx"
- board text added: "SIG"
- board text added: "Tx"
- board text added: "VESC BRAIN BOARD V1.0"
- board text added: "Vcc"
