File: brainboardV1.0/VESC_brain_board.kicad_sch (KiCad schematic)
At the start: 19 parts, among them J1 Conn_01x18, J2 Conn_01x04, Q1 my_BC337, U2 TJA1050T/CM,118, U2 Teensy4.0

Commit message: finished V1.0
Parts:
- removed R3 (x2): 10k, Resistor_SMD:R_0603_1608Metric, symbol Device:R
- 1k_1: footprint Resistor_SMD:R_0805_2012Metric -> Resistor_SMD:R_0603_1608Metric
- DC_2: footprint Capacitor_SMD:C_0805_2012Metric -> Capacitor_SMD:C_0603_1608Metric
Connections:
- net BUTTON: now also U2.24 (17_A3_TX4_SDA1)
- net SPEAKER: now also U2.20 (13_SCK_CRX1_LED)
- net VESC1_TX: now also U2.14 (12_MISO_MQSL)
- net VESC2_ADC2: now also U2.22 (15_A1_RX3_SPDIF_IN)
- net VESC2_EN: now also U2.21 (14_A0_TX3_SPDIF_OUT)
- net VESC2_TX: now also U2.23 (16_A2_RX4_SCL1)
- net VSENSE: now also U2.28 (21_A7_RX5_BCLK1); no longer U2.21 (14_A0_TX3_SPDIF_OUT)
- no-connect marks 18 -> 19
Other:
- note removed: "doublecheck pinouts of transistor"
