File: brainboardV1.0/MESC_brain_board.kicad_pcb (KiCad board)
At the start: 4 copper layers, 90.5 x 68.6 mm, 54 parts, among them J1 Conn_01x18, J12 Conn_01x03, J13 Conn_01x03, J14 SERIAL1, J15 Conn_01x03, J21 Conn_01x01, J22 Conn_01x01, J23 Conn_01x01, Q1 my_BC337, U1 TJA1050T/CM,118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

Commit message: finalized PCB, changed file names
Parts:
- removed J21, J23: Conn_01x01, Connector_PinSocket_2.54mm:PinSocket_1x01_P2.54mm_Vertical
- added J24: Conn_01x01, Connector_Wire:SolderWire-2sqmm_1x01_D2mm_OD3.9mm, F.Cu at (99.2, 80.2)
- added J25: Conn_01x01, Connector_Wire:SolderWire-2sqmm_1x01_D2mm_OD3.9mm, F.Cu at (93.8, 80.2)
- added U22: my_buck_boost, Converter_DCDC:my_buck_boost, F.Cu at (94.0, 65.5)
- moved J22 68.3 mm to (43.0, 29.8)
- moved REF** 12.2 mm to (80.5, 72.8)
- moved MESC1 2.65 mm to (64.8, 80.5)
- moved MESC2 2.65 mm to (86.8, 80.7)
- moved 10k_8 2.39 mm to (69.8, 60.9)
- moved DC_1 2.39 mm to (79.4, 65.9)
- moved S1 2.39 mm to (74.0, 66.0)
- moved SW_SPDT21 2.33 mm to (22.5, 29.8)
- moved REF** 1.46 mm to (41.8, 77.5)
- renumbered VESC1 to MESC1, VESC2 to MESC2
Connections:
- net VESC1_ADC1 renamed MESC1_ADC1
- net VESC1_ADC2 renamed MESC1_ADC2
- net VESC1_EN renamed MESC1_EN
- net VESC1_RX renamed MESC1_RX
- net VESC1_TX renamed MESC1_TX
- net VESC1_VCC renamed MESC1_VCC
- net VESC2_ADC1 renamed MESC2_ADC1
- net VESC2_ADC2 renamed MESC2_ADC2
- net VESC2_EN renamed MESC2_EN
- net VESC2_RX renamed MESC2_RX
- net VESC2_TX renamed MESC2_TX
- net VESC2_VCC renamed MESC2_VCC
- MESC1 pad 1: VESC_+5V -> MESC1_+5V
- MESC2 pad 1: VESC_+5V -> MESC2_+5V
- SW_SPDT21 pad 1: +5V -> Net-(SW_SPDT21-A)
- SW_SPDT21 pad 2: VESC_+5V -> Vcc
Routing:
- net Net-(SW_SPDT21-A): track 0.00 -> 149.7 mm
- net Vcc: track 0.00 -> 135.7 mm
- net VESC_+5V: track 130.1 -> 0.00 mm
- net +5V: track 281.5 -> 329.0 mm, vias 6 -> 7
- net GND: track 45.6 -> 50.7 mm
- net MESC2_ADC2: track 42.4 -> 38.1 mm
- net MESC1_ADC2: track 41.3 -> 37.5 mm
- net MESC1_EN: track 43.4 -> 39.6 mm
- net MESC2_EN: track 37.8 -> 34.1 mm
- net MESC1_TX: track 40.4 -> 37.0 mm
- net MESC2_TX: track 45.4 -> 42.3 mm
- net MESC1_VCC: track 122.4 -> 120.0 mm
- net BUTTON: track 35.5 -> 34.3 mm
Other:
- board text added: "MESC BRAIN BOARD V1.0"
- board text added: "MESC1"
- board text added: "MESC2"
- board text added: "RC Tx/Rx"
- board text removed: "VESC BRAIN BOARD V1.0"

Commit message: finalizing PCB
Parts:
- MESC1, MESC2: value Conn_01x08 -> Conn_01x06; footprint Connector_JST:JST_PH_B8B-PH-K_1x08_P2.00mm_Vertical -> Connector_JST:JST_PH_B6B-PH-K_1x06_P2.00mm_Vertical
- moved MESC1 4.26 mm to (60.5, 80.8)
- moved MESC2 4.00 mm to (82.8, 80.8)
Connections:
- MESC1 pad 1: MESC1_+5V -> unconnected-(MESC1-Pin_1-Pad1)
- MESC1 pad 2: MESC1_VCC -> GND
- MESC1 pad 3: GND -> PB6_1
- MESC1 pad 4: MESC1_ADC1 -> PB5_1
- MESC1 pad 5: MESC1_RX -> PB4_1
- MESC1 pad 6: MESC1_TX -> PB3_1
- MESC2 pad 1: MESC2_+5V -> unconnected-(MESC2-Pin_1-Pad1)
- MESC2 pad 2: MESC2_VCC -> GND
- MESC2 pad 3: GND -> PB6_2
- MESC2 pad 4: MESC2_ADC1 -> PB5_2
- MESC2 pad 5: MESC2_RX -> PB4_2
- MESC2 pad 6: MESC2_TX -> PB3_2
- U2 pad 12: MESC1_EN -> PB3_1
- U2 pad 13: MESC1_ADC2 -> PB4_1
- U2 pad 14: MESC1_TX -> PB5_1
- U2 pad 21: MESC2_EN -> PB3_2
- U2 pad 22: MESC2_ADC2 -> PB4_2
- U2 pad 23: MESC2_TX -> PB5_2
Routing:
- net MESC1_VCC: track 120.0 -> 2.18 mm, vias 2 -> 1
- net PB5_2: track 0.00 -> 42.3 mm
- net MESC2_TX: track 42.3 -> 0.00 mm
- net MESC1_EN: track 39.6 -> 0.00 mm
- net PB3_1: track 0.00 -> 39.3 mm
- net PB4_2: track 0.00 -> 38.1 mm
- net MESC2_ADC2: track 38.1 -> 0.00 mm
- net MESC1_ADC2: track 37.5 -> 0.00 mm
- net PB4_1: track 0.00 -> 37.2 mm
- net MESC1_TX: track 37.0 -> 0.00 mm
- net PB5_1: track 0.00 -> 36.7 mm
- net PB3_2: track 0.00 -> 34.1 mm
- net MESC2_EN: track 34.1 -> 0.00 mm
Other:
- board text added: "<16v only!!"
- board text added: "PB3"
- board text added: "PB4"
- board text added: "PB5"

Commit message: First board ordered from JLCPCB
Connections:
- MESC1 pad 1: unconnected-(MESC1-Pin_1-Pad1) -> +5V
- MESC2 pad 1: unconnected-(MESC2-Pin_1-Pad1) -> +5V
Routing:
- net +5V: track 329.0 -> 365.8 mm, vias 7 -> 8
- net /CAN_RX: track 30.6 -> 29.3 mm
- net GND: vias 13 -> 17
Other:
- board text added: "ESP32 PROG"
- board text added: "ESP32-WROOM-32D"
- board text added: "MESC input MUST be set to +5V"
- board text added: "NC"
- board text added: "Not implemented"
- board text added: "TEENSY4.0"
