File: brainboardV1.0/MESC_brain_board.kicad_sch (KiCad schematic)
At the start: 17 parts, among them J1 Conn_01x18, J2 Conn_01x04, Q1 my_BC337, U2 TJA1050T/CM,118, U2 Teensy4.0

Commit message: finalized PCB, changed file names
Parts:
- renumbered VESC1 to MESC1, VESC2 to MESC2
Connections:
- net VESC1_ADC1 renamed MESC1_ADC1
- net VESC1_ADC2 renamed MESC1_ADC2
- net VESC1_EN renamed MESC1_EN
- net VESC1_RX renamed MESC1_RX
- net VESC1_TX renamed MESC1_TX
- net VESC1_VCC renamed MESC1_VCC
- net VESC2_ADC1 renamed MESC2_ADC1
- net VESC2_ADC2 renamed MESC2_ADC2
- net VESC2_EN renamed MESC2_EN
- net VESC2_RX renamed MESC2_RX
- net VESC2_TX renamed MESC2_TX
- net VESC2_VCC renamed MESC2_VCC
- net VESC_+5V renamed MESC1_+5V
- net MESC1_+5V: no longer MESC2.1 (Pin_1)
- new net MESC2_+5V: MESC2.1 (Pin_1)
Other:
- note added: "MESC I/O Reserved 2 GPIO pins on Teensy for emergency shutoff to MESC CAN connector (for MESC motor control) Voltage divider (to monitor battery voltage)"
- note removed: "VESC I/O Reserved 2 GPIO pins on Teensy for emergency shutoff to VESC CAN connector (for VESC motor control) Voltage divider (to monitor battery voltage)"
Changed lines of the file:
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@@
 		)
 	)
-	(text "VESC I/O\nReserved 2 GPIO pins on Teensy for emergency shutoff to VESC\nCAN connector (for VESC motor control)\nVoltage divider (to monitor battery voltage)\n\n"
+	(text "MESC I/O\nReserved 2 GPIO pins on Teensy for emergency shutoff to MESC\nCAN connector (for MESC motor control)\nVoltage divider (to monitor battery voltage)\n\n"
 		(exclude_from_sim no)
 		(at 165.1 141.224 0)
@@
 		)
 	)
-	(label "VESC1_TX"
+	(label "MESC1_TX"
 		(at 154.94 52.07 0)
 		(effects
@@
 		)
 	)
-	(label "VESC1_EN"
+	(label "MESC1_EN"
 		(at 154.94 46.99 0)
 		(effects
@@
 		)
 	)
-	(label "VESC2_EN"
+	(label "MESC2_EN"
 		(at 154.94 69.85 0)
 		(effects
@@
 		)
 	)
-	(label "VESC1_ADC2"
+	(label "MESC1_ADC2"
 		(at 154.94 49.53 0)
 		(effects
@@
 		)
 	)
-	(label "VESC2_TX"
+	(label "MESC2_TX"
 		(at 154.94 74.93 0)
 		(effects
@@
 		)
 	)
-	(label "VESC2_ADC2"
+	(label "MESC2_ADC2"
 		(at 154.94 72.39 0)
 		(effects
@@
 		)
 	)
-	(global_label "VESC2_ADC2"
+	(global_label "MESC2_ADC2"
 		(shape input)
 		(at 70.485 158.115 180)
@@
 		)
 	)
-	(global_label "VESC1_EN"
+	(global_label "MESC1_EN"
 		(shape input)
 		(at 70.485 137.795 180)
@@
 		)
 	)
-	(global_label "VESC1_RX"
+	(global_label "MESC1_RX"
 		(shape input)
 		(at 70.485 130.175 180)
@@
 		)
 	)
-	(global_label "VESC1_ADC2"
+	(global_label "MESC1_ADC2"
 		(shape input)
 		(at 70.485 135.255 180)
@@
 		)
 	)
-	(global_label "VESC2_EN"
+	(global_label "MESC2_EN"
 		(shape input)
 		(at 70.485 160.655 180)
@@
 		)
 	)
-	(global_label "VESC1_TX"
+	(global_label "MESC1_TX"
 		(shape input)
 		(at 70.485 132.715 180)
@@
 		)
 	)
-	(global_label "VESC2_TX"
+	(global_label "MESC2_TX"
 		(shape input)
 		(at 70.485 155.575 180)
@@
 		)
 	)
-	(global_label "VESC2_RX"
+	(global_label "MESC2_RX"
 		(shape input)
 		(at 70.485 153.035 180)
@@
 		)
 	)
-	(global_label "VESC2_VCC"
+	(global_label "MESC2_VCC"
 		(shape input)
 		(at 70.485 145.415 180)
@@
 		)
 	)
-	(global_label "VESC_+5V"
+	(global_label "MESC1_+5V"
 		(shape input)
 		(at 70.485 120.015 180)
@@
 		)
 		(property "Intersheetrefs" "${INTERSHEET_REFS}"
-			(at 57.9446 120.015 0)
+			(at 56.7351 120.015 0)
 			(effects
 				(font
@@
 		)
 	)
-	(global_label "VESC_+5V"
+	(global_label "MESC2_+5V"
 		(shape input)
 		(at 70.485 142.875 180)
@@
 		)
 		(property "Intersheetrefs" "${INTERSHEET_REFS}"
-			(at 57.9446 142.875 0)
+			(at 56.7351 142.875 0)
 			(effects
 				(font
@@
 		)
 	)
-	(global_label "VESC1_VCC"
+	(global_label "MESC1_VCC"
 		(shape input)
 		(at 70.485 122.555 180)
@@
 		)
 	)
-	(global_label "VESC1_ADC1"
+	(global_label "MESC1_ADC1"
 		(shape input)
 		(at 70.485 127.635 180)
@@
 		)
 	)
-	(global_label "VESC2_ADC1"
+	(global_label "MESC2_ADC1"
 		(shape input)
 		(at 70.485 150.495 180)
@@
 		)
 		(instances
-			(project "VESC_brain_board"
+			(project "MESC_brain_board"
 				(path "/8920b97c-b80b-47c5-aaa4-fe68c48cd11a"
 					(reference "JP1")
@@
 				)
 			)
-			(project "VESC_brain_board"
+			(project "MESC_brain_board"
 				(path "/8920b97c-b80b-47c5-aaa4-fe68c48cd11a"
 					(reference "R_120")
@@
 		)
 		(instances
-			(project "VESC_brain_board"
+			(project "MESC_brain_board"
 				(path "/8920b97c-b80b-47c5-aaa4-fe68c48cd11a"
 					(reference "U2")
@@
 		)
 		(instances
-			(project "VESC_brain_board"
+			(project "MESC_brain_board"
 				(path "/8920b97c-b80b-47c5-aaa4-fe68c48cd11a"
 					(reference "Q1")
@@
 		)
 		(instances
-			(project "VESC_brain_board"
+			(project "MESC_brain_board"
 				(path "/8920b97c-b80b-47c5-aaa4-fe68c48cd11a"
 					(reference "#PWR012")
@@
 				)
 			)
-			(project "VESC_brain_board"
+			(project "MESC_brain_board"
 				(path "/8920b97c-b80b-47c5-aaa4-fe68c48cd11a"
 					(reference "10k_1")
@@
 		)
 		(instances
-			(project "VESC_brain_board"
+			(project "MESC_brain_board"
 				(path "/8920b97c-b80b-47c5-aaa4-fe68c48cd11a"
 					(reference "#PWR026")
@@
 		)
 		(instances
-			(project "VESC_brain_board"
+			(project "MESC_brain_board"
 				(path "/8920b97c-b80b-47c5-aaa4-fe68c48cd11a"
 					(reference "S1")
@@
 		)
 		(instances
-			(project "VESC_brain_board"
+			(project "MESC_brain_board"
 				(path "/8920b97c-b80b-47c5-aaa4-fe68c48cd11a"
 					(reference "10k_8")
@@
 				)
 			)
-			(project "VESC_brain_board"
+			(project "MESC_brain_board"
 				(path "/8920b97c-b80b-47c5-aaa4-fe68c48cd11a"
 					(reference "U1")
@@
 		)
 		(instances
-			(project "VESC_brain_board"
+			(project "MESC_brain_board"
 				(path "/8920b97c-b80b-47c5-aaa4-fe68c48cd11a"
 					(reference "DC_1")
@@
 		)
 		(instances
-			(project "VESC_brain_board"
+			(project "MESC_brain_board"
 				(path "/8920b97c-b80b-47c5-aaa4-fe68c48cd11a"
 					(reference "DC_2")
@@
 		)
 		(instances
-			(project "VESC_brain_board"
+			(project "MESC_brain_board"
 				(path "/8920b97c-b80b-47c5-aaa4-fe68c48cd11a"
 					(reference "#PWR03")
@@
 		(dnp no)
 		(fields_autoplaced yes)
-		(property "Reference" "VESC2"
+		(property "Reference" "MESC2"
 			(at 78.105 151.7649 0)
 			(effects
@@
 		)
 		(instances
-			(project "VESC_brain_board"
+			(project "MESC_brain_board"
 				(path "/8920b97c-b80b-47c5-aaa4-fe68c48cd11a"
-					(reference "VESC2")
+					(reference "MESC2")
 					(unit 1)
 				)
@@
 		)
 		(instances
-			(project "VESC_brain_board"
+			(project "MESC_brain_board"
 				(path "/8920b97c-b80b-47c5-aaa4-fe68c48cd11a"
 					(reference "MP1")
@@
 				)
 			)
-			(project "VESC_brain_board"
+			(project "MESC_brain_board"
 				(path "/8920b97c-b80b-47c5-aaa4-fe68c48cd11a"
 					(reference "CAN1")
@@
 		)
 		(instances
-			(project "VESC_brain_board"
+			(project "MESC_brain_board"
 				(path "/8920b97c-b80b-47c5-aaa4-fe68c48cd11a"
 					(reference "1k_1")
@@
 		)
 		(instances
-			(project "VESC_brain_board"
+			(project "MESC_brain_board"
 				(path "/8920b97c-b80b-47c5-aaa4-fe68c48cd11a"
 					(reference "LS1")
@@
 		(dnp no)
 		(fields_autoplaced yes)
-		(property "Reference" "VESC1"
+		(property "Reference" "MESC1"
 			(at 78.105 128.9049 0)
 			(effects
@@
 			(project ""
 				(path "/8920b97c-b80b-47c5-aaa4-fe68c48cd11a"
-					(reference "VESC1")
+					(reference "MESC1")
 					(unit 1)
 				)
@@
 		)
 		(instances
-			(project "VESC_brain_board"
+			(project "MESC_brain_board"
 				(path "/8920b97c-b80b-47c5-aaa4-fe68c48cd11a"
 					(reference "#PWR027")
@@
 		)
 		(instances
-			(project "VESC_brain_board"
+			(project "MESC_brain_board"
 				(path "/8920b97c-b80b-47c5-aaa4-fe68c48cd11a"
 					(page "3")
@@
 		)
 		(instances
-			(project "VESC_brain_board"
+			(project "MESC_brain_board"
 				(path "/8920b97c-b80b-47c5-aaa4-fe68c48cd11a"
 					(page "2")

Commit message: finalizing PCB
Parts:
- removed MESC1, MESC2: Conn_01x08, Connector_JST:JST_PH_B8B-PH-K_1x08_P2.00mm_Vertical, symbol Connector_Generic:Conn_01x08
- added MESC1, MESC2: Conn_01x06, Connector_JST:JST_PH_B6B-PH-K_1x06_P2.00mm_Vertical, symbol Connector_Generic:Conn_01x06
Connections:
- net GND: now also MESC1.2 (Pin_2), MESC2.2 (Pin_2)
- net MESC1_ADC2 renamed PB4_1
- net PB4_1: now also MESC1.5 (Pin_5)
- net MESC1_EN renamed PB3_1
- net PB3_1: now also MESC1.6 (Pin_6)
- net MESC1_TX renamed PB5_1
- net PB5_1: now also MESC1.4 (Pin_4)
- net MESC2_ADC2 renamed PB4_2
- net PB4_2: now also MESC2.5 (Pin_5)
- net MESC2_EN renamed PB3_2
- net PB3_2: now also MESC2.6 (Pin_6)
- net MESC2_TX renamed PB5_2
- net PB5_2: now also MESC2.4 (Pin_4)
- new net PB6_1: MESC1.3 (Pin_3)
- new net PB6_2: MESC2.3 (Pin_3)
- no-connect marks 19 -> 21
Other:
- moved on the sheet: J1

Commit message: First board ordered from JLCPCB
Connections:
- net +5V: now also MESC1.1 (Pin_1), MESC2.1 (Pin_1)
Other:
- note added: "Not great design w/ DC-DC conversion from high voltage VBat"
