File: MT6701_ENCODER/MT6701_ENCODER.kicad_pcb (KiCad board)
At the start: 4 copper layers, 20.8 x 15.7 mm, 9 parts, among them J5 Conn_01x05, U1 MT6701CT

Commit message: used for jlcpcb
Parts:
- added REF**: MountingHole_4.3mm_M4, MountingHole:MountingHole_4.3mm_M4, F.Cu at (115.0, 100.0)
- added REF**: MountingHole_4.3mm_M4, MountingHole:MountingHole_4.3mm_M4, F.Cu at (85.0, 100.0)
- J5: moved to B.Cu
- moved J5 119.2 mm to (105.1, 108.1)
- moved JP2 111.2 mm to (105.8, 100.0)
- moved R1 111.2 mm to (97.7, 103.7)
- moved R2 111.2 mm to (102.3, 103.7)
- moved TVS1 111.2 mm to (95.0, 102.2)
- moved C1 111.2 mm to (95.5, 98.8)
- moved JP1 111.2 mm to (105.8, 102.7)
- moved JP3 111.2 mm to (100.0, 100.3)
- moved U1 111.2 mm to (100.0, 100.0)
Routing:
- net Vcc: track 12.8 -> 10.2 mm, vias 0 -> 2
- net ENC_Z: track 10.7 -> 13.0 mm
- net ENC_A: track 11.9 -> 13.3 mm
- net GND: track 7.22 -> 6.21 mm, vias 2 -> 1
Other:
- board size 20.8 x 15.7 mm -> 38.4 x 30 mm
- board text added: "30mm"
- board text added: "MT6701 ENCODER V1.0"
- board text added: "SCL"
- board text added: "SDA"
