File: PCBs/brainboardV1.4/CAN.kicad_sch (KiCad schematic)
At the start: 10 parts, among them U22 TCAN332GDCNT

Commit message: finalization of BB V1.4
Connections:
- net CAN_CM_BIAS: no longer names the net of C21.1, R60_21.1, R60_22.2
- net CAN_CM_BIAS: no longer U22.5 (Vref)
- no-connect marks 0 -> 1
Changed lines of the file:
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@@
-	)
-	(junction
-		(at 139.7 90.17)
-		(diameter 0)
-		(color 0 0 0 0)
 	)
 	(junction
@@
 		(color 0 0 0 0)
 	)
+	(no_connect
+		(at 161.29 78.74)
+	)
 	(wire
 		(pts
@@
 	(wire
 		(pts
-			(xy 161.29 78.74) (xy 167.64 78.74)
-		)
-		(stroke
-			(width 0)
-			(type default)
-		)
-	)
-	(wire
-		(pts
 			(xy 167.64 60.96) (xy 165.1 60.96)
 		)
@@
 	(wire
 		(pts
-			(xy 139.7 90.17) (xy 140.97 90.17)
-		)
-		(stroke
-			(width 0)
-			(type default)
-		)
-	)
-	(wire
-		(pts
 			(xy 165.1 91.44) (xy 165.1 93.98)
 		)
@@
 	(wire
 		(pts
-			(xy 139.7 90.17) (xy 139.7 92.71)
-		)
-		(stroke
-			(width 0)
-			(type default)
-		)
-	)
-	(wire
-		(pts
-			(xy 139.7 85.09) (xy 139.7 90.17)
+			(xy 139.7 85.09) (xy 139.7 92.71)
 		)
 		(stroke
@@
 		)
 	)
-	(global_label "CAN_CM_BIAS"
-		(shape input)
-		(at 140.97 90.17 0)
+	(global_label "+3.3V"
+		(shape input)
+		(at 148.59 66.04 180)
+		(fields_autoplaced yes)
+		(effects
+			(font
+				(size 1.27 1.27)
+			)
+			(justify right)
+		)
+		(property "Intersheetrefs" "${INTERSHEET_REFS}"
+			(at 139.92 66.04 0)
+			(effects
+				(font
+					(size 1.27 1.27)
+				)
+				(justify right)
+				(hide yes)
+			)
+		)
+	)
+	(global_label "+3.3V"
+		(shape input)
+		(at 167.64 93.98 0)
 		(fields_autoplaced yes)
 		(effects
@@
 		)
 		(property "Intersheetrefs" "${INTERSHEET_REFS}"
-			(at 156.4738 90.17 0)
+			(at 176.31 93.98 0)
 			(effects
 				(font
@@
 		)
 	)
-	(global_label "+3.3V"
-		(shape input)
-		(at 148.59 66.04 180)
+	(global_label "CAN_HI"
+		(shape input)
+		(at 115.57 76.2 180)
 		(fields_autoplaced yes)
 		(effects
@@
 		)
 		(property "Intersheetrefs" "${INTERSHEET_REFS}"
-			(at 139.92 66.04 0)
+			(at 106.7264 76.2 0)
 			(effects
 				(font
@@
 		)
 	)
-	(global_label "+3.3V"
-		(shape input)
-		(at 167.64 93.98 0)
+	(global_label "CAN_LO"
+		(shape input)
+		(at 115.57 83.82 180)
+		(fields_autoplaced yes)
+		(effects
+			(font
+				(size 1.27 1.27)
+			)
+			(justify right)
+		)
+		(property "Intersheetrefs" "${INTERSHEET_REFS}"
+			(at 106.3031 83.82 0)
+			(effects
+				(font
+					(size 1.27 1.27)
+				)
+				(justify right)
+				(hide yes)
+			)
+		)
+	)
+	(global_label "GND"
+		(shape input)
+		(at 140.97 101.6 0)
 		(fields_autoplaced yes)
 		(effects
@@
 		)
 		(property "Intersheetrefs" "${INTERSHEET_REFS}"
-			(at 176.31 93.98 0)
+			(at 147.0921 101.6 0)
 			(effects
 				(font
@@
 		)
 	)
+	(global_label "CAN_STB"
+		(shape input)
+		(at 167.64 81.28 0)
+		(fields_autoplaced yes)
+		(effects
+			(font
+				(size 1.27 1.27)
+			)
+			(justify left)
+		)
+		(property "Intersheetrefs" "${INTERSHEET_REFS}"
+			(at 178.729 81.28 0)
+			(effects
+				(font
+					(size 1.27 1.27)
+				)
+				(justify left)
+				(hide yes)
+			)
+		)
+	)
 	(global_label "CAN_HI"
 		(shape input)
-		(at 115.57 76.2 180)
+		(at 97.79 101.6 180)
 		(fields_autoplaced yes)
 		(effects
@@
 		)
 		(property "Intersheetrefs" "${INTERSHEET_REFS}"
-			(at 106.7264 76.2 0)
+			(at 88.9464 101.6 0)
 			(effects
 				(font
@@
 				(hide yes)
 			)
-		)
-	)
-	(global_label "CAN_LO"
-		(shape input)
-		(at 115.57 83.82 180)
-		(fields_autoplaced yes)
-		(effects
-			(font
-				(size 1.27 1.27)
-			)
-			(justify right)
-		)
-		(property "Intersheetrefs" "${INTERSHEET_REFS}"
-			(at 106.3031 83.82 0)
-			(effects
-				(font
-					(size 1.27 1.27)
-				)
-				(justify right)
-				(hide yes)
-			)
-		)
-	)
-	(global_label "GND"
-		(shape input)
-		(at 140.97 101.6 0)
-		(fields_autoplaced yes)
-		(effects
-			(font
-				(size 1.27 1.27)
-			)
-			(justify left)
-		)
-		(property "Intersheetrefs" "${INTERSHEET_REFS}"
-			(at 147.0921 101.6 0)
-			(effects
-				(font
-					(size 1.27 1.27)
-				)
-				(justify left)
-				(hide yes)
-			)
-		)
-	)
-	(global_label "CAN_STB"
-		(shape input)
-		(at 167.64 81.28 0)
-		(fields_autoplaced yes)
-		(effects
-			(font
-				(size 1.27 1.27)
-			)
-			(justify left)
-		)
-		(property "Intersheetrefs" "${INTERSHEET_REFS}"
-			(at 178.729 81.28 0)
-			(effects
-				(font
-					(size 1.27 1.27)
-				)
-				(justify left)
-				(hide yes)
-			)
-		)
-	)
-	(global_label "CAN_HI"
-		(shape input)
-		(at 97.79 101.6 180)
-		(fields_autoplaced yes)
-		(effects
-			(font
-				(size 1.27 1.27)
-			)
-			(justify right)
-		)
-		(property "Intersheetrefs" "${INTERSHEET_REFS}"
-			(at 88.9464 101.6 0)
-			(effects
-				(font
-					(size 1.27 1.27)
-				)
-				(justify right)
-				(hide yes)
-			)
-		)
-	)
-	(global_label "CAN_CM_BIAS"
-		(shape input)
-		(at 167.64 78.74 0)
-		(fields_autoplaced yes)
-		(effects
-			(font
-				(size 1.27 1.27)
-			)
-			(justify left)
-		)
-		(property "Intersheetrefs" "${INTERSHEET_REFS}"
-			(at 183.1438 78.74 0)
-			(effects
-				(font
-					(size 1.27 1.27)
-				)
-				(justify left)
-				(hide yes)
-			)

Commit message: updated brainboard v1.4
Parts:
- C21: P/N 810-C2012X7R2A104K -> CC0603JRNPO9BN472
- U22: value TCAN332GDCNT -> TCAN334GDR
Other:
- note added: "CAN NODE DESIGN NOTES - TEENSY 4.0 + TCAN334G • 3.3 V CAN transceiver w/ standby (TCAN334G must be used) • VCC = 3.3 V with local 0.1 µF decoupling at device • TXD pull-up to 3.3 V (10k) → recessive during MCU reset • STB pull-up to 3.3 V (10k) → default standby; MCU drives LOW after FlexCAN init • Direct MCU interface: TXD↔CAN_TX, RXD↔CAN_RX (no level shifting) • VREF not used (leave NC) • Split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"
- note removed: "CAN NODE DESIGN NOTES - TEENSY 4.0 + TCAN332G • 3.3 V CAN transceiver w/ standby (TCAN332G) • VCC = 3.3 V with local 0.1 µF decoupling at device • TXD pull-up to 3.3 V (10k) → recessive during MCU reset • STB pull-up to 3.3 V (10k) → default standby; MCU drives LOW after FlexCAN init • Direct MCU interface: TXD↔CAN_TX, RXD↔CAN_RX (no level shifting) • VREF not used (leave NC) • Split termination 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"
Changed lines of the file:
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@@
 	(generator_version "9.0")
 	(paper "A4")
-	(text "CAN NODE DESIGN NOTES - TEENSY 4.0 + TCAN332G\n• 3.3 V CAN transceiver w/ standby (TCAN332G)\n• VCC = 3.3 V with local 0.1 µF decoupling at device\n• TXD pull-up to 3.3 V (10k) → recessive during MCU reset\n• STB pull-up to 3.3 V (10k) → default standby; MCU drives LOW after FlexCAN init\n• Direct MCU interface: TXD↔CAN_TX, RXD↔CAN_RX (no level shifting)\n• VREF not used (leave NC)\n• Split termination 2, 60Ω termination only at physical bus ends\n• CAN TVS (SM24CANB-02) at connector; hot plug protection"
+	(text "CAN NODE DESIGN NOTES - TEENSY 4.0 + TCAN334G\n• 3.3 V CAN transceiver w/ standby (TCAN334G must be used)\n• VCC = 3.3 V with local 0.1 µF decoupling at device\n• TXD pull-up to 3.3 V (10k) → recessive during MCU reset\n• STB pull-up to 3.3 V (10k) → default standby; MCU drives LOW after FlexCAN init\n• Direct MCU interface: TXD↔CAN_TX, RXD↔CAN_RX (no level shifting)\n• VREF not used (leave NC)\n• Split termination 2, 60Ω termination only at physical bus ends\n• CAN TVS (SM24CANB-02) at connector; hot plug protection"
 		(exclude_from_sim no)
 		(at 116.586 115.57 0)
@@
 			)
 		)
-		(property "Datasheet" "https://www.mouser.com/ProductDetail/TDK/C2012X7R2A104K125AA?qs=NRhsANhppD9J0ZsT2%2Fo%2F7Q%3D%3D"
+		(property "Datasheet" ""
 			(at 139.7 96.52 0)
 			(effects
@@
 			)
 		)
-		(property "P/N" "810-C2012X7R2A104K"
+		(property "P/N" "CC0603JRNPO9BN472"
 			(at 139.7 96.52 0)
 			(effects
@@
 			)
 		)
-		(property "Value" "TCAN332GDCNT"
+		(property "Value" "TCAN334GDR"
 			(at 164.338 61.468 0)
 			(effects
