File: PCBs/brainboardV1.4/MESC_brain_board.kicad_pcb (KiCad board)
At the start: 4 copper layers, 84.5 x 64 mm, 53 parts, among them J1 Conn_01x18, J12 Conn_01x03, J13 Conn_01x03, J14 SERIAL1, J15 Conn_01x03, J21 Conn_01x07, J22 Conn_01x01, J23 Conn_01x01, J24 Conn_01x01, J25 Conn_01x01, Q1 my_BC337, U1 TJA1050T/CM,118, U11 ESP32-WROOM-32D, U2 Teensy4.0, U21 LD1117S18TR_SOT223, U24 12_DCDC_5

Commit message: brain board V1.4
Parts:
- removed 10k_1, 10k_4, 10k_5, 10k_8: 10k, Resistor_SMD:R_0603_1608Metric
- removed the 1k_21 at (71.0, 59.0)
- removed 1k_22: 1k, Resistor_SMD:R_0603_1608Metric
- removed 20k_1, R20k_4: 20k, Resistor_SMD:R_0603_1608Metric
- removed 5k_2: 5k, Resistor_SMD:R_0603_1608Metric
- removed DC_1, DC_3, DC_4, DC_6: 100nF, Capacitor_SMD:C_0603_1608Metric
- removed DC_5: 10uF, Capacitor_SMD:C_0805_2012Metric
- removed D_BLU2: BLUE, LED_SMD:LED_0603_1608Metric
- removed D_GRN1: LED GRN, LED_SMD:LED_0603_1608Metric
- removed D_RED1: LED RED, LED_SMD:LED_0603_1608Metric
- removed J12, J13, J15: Conn_01x03, Connector_PinHeader_2.54mm:PinHeader_1x03_P2.54mm_Vertical
- removed J14: SERIAL1, Connector_PinHeader_2.54mm:PinHeader_1x04_P2.54mm_Vertical
- removed JP1: SolderJumper_3_Open, Jumper:SolderJumper-3_P1.3mm_Open_Pad1.0x1.5mm
- removed the REF** at (96.7, 23.7)
- removed the REF** at (20.1, 23.7)
- removed the REF** at (96.7, 80.1)
- removed the REF** at (20.1, 80.1)
- removed R_120: 120, Resistor_SMD:R_0603_1608Metric
- removed S1: TL3342F160QG, Button_Switch_SMD:SW_SPST_B3SL-1022P
- removed S11, S12: TL3342F160QG, Button_Switch_SMD:SW_Push_SPST_NO_Alps_SKRK
- removed U1: TJA1050T/CM,118, Package_SO:SOIC-8_3.9x4.9mm_P1.27mm
- removed U11: ESP32-WROOM-32D, RF_Module:ESP32-WROOM-32D
- added 10k_11: 10k, Resistor_SMD:R_0603_1608Metric, F.Cu at (50.1, 58.9)
- added 10k_22: 10k, Resistor_SMD:R_0603_1608Metric, F.Cu at (86.0, 48.5)
- added 10k_23: 10k, Resistor_SMD:R_0603_1608Metric, F.Cu at (86.7, 53.4)
- added 20k_21: 20k, Resistor_SMD:R_0603_1608Metric, F.Cu at (83.7, 22.9)
- added 5k_21: 5k, Resistor_SMD:R_0603_1608Metric, F.Cu at (77.1, 22.8)
- added C21: 4.7nF, Capacitor_SMD:C_0603_1608Metric, F.Cu at (82.5, 57.6)
- added D21: SM24CANB-02HTG, SM24CANB-02HTG:SOT95P230X117-3N, F.Cu at (82.3, 61.0)
- added DC_12: 100nF, Capacitor_SMD:C_0603_1608Metric, F.Cu at (28.6, 69.8)
- added DC_23: 100nF, Capacitor_SMD:C_0603_1608Metric, F.Cu at (82.6, 46.2)
- added D_GRN21: LED GRN, LED_SMD:LED_0603_1608Metric, F.Cu at (77.0, 24.4)
- added D_RED21: LED RED, LED_SMD:LED_0603_1608Metric, F.Cu at (83.6, 24.4)
- added ESP1: Conn_01x04, Connector_JST:JST_PH_B4B-PH-K_1x04_P2.00mm_Vertical, F.Cu at (62.3, 59.2)
- added R60_21: 60, Resistor_SMD:R_0603_1608Metric, F.Cu at (84.3, 57.6)
- added R60_22: 60, Resistor_SMD:R_0603_1608Metric, F.Cu at (80.8, 57.5)
- added REF**: MountingHole_3.2mm_M3, MountingHole:MountingHole_3.2mm_M3, F.Cu at (96.9, 23.8)
- added REF**: MountingHole_3.2mm_M3, MountingHole:MountingHole_3.2mm_M3, F.Cu at (20.4, 23.8)
- added REF**: MountingHole_3.2mm_M3, MountingHole:MountingHole_3.2mm_M3, F.Cu at (96.9, 80.2)
- added REF**: MountingHole_3.2mm_M3, MountingHole:MountingHole_3.2mm_M3, F.Cu at (20.4, 80.2)
- added S21: TL3342F160QG, Button_Switch_SMD:SW_Push_SPST_NO_Alps_SKRK, F.Cu at (28.9, 75.3)
- added TP21: TestPoint, Connector_PinSocket_2.54mm:PinSocket_1x01_P2.54mm_Vertical, F.Cu at (79.9, 73.3)
- added TP22: TestPoint, Connector_PinSocket_2.54mm:PinSocket_1x01_P2.54mm_Vertical, F.Cu at (83.7, 73.3)
- added U22: TCAN332GDCNT, Package_SO:SOIC-8_3.9x4.9mm_P1.27mm, F.Cu at (82.5, 50.9)
- moved CAN1 33.8 mm to (85.2, 66.3), turned to 180 degrees
- moved C25 0.72 mm to (57.0, 77.9)
- moved J26 0.52 mm to (51.4, 79.8)
- renumbered 1k_1 to 1k_21, 20k_21 to 20k_22, C21 to C22, C25 to C23, C27 to C24, C23 to C25, DC_2 to DC_21, MESC1 to GPIO1, J21 to IMU1, J22 to J24, J24 to J26, LS1 to LS21, Q1 to Q21, U2 to U21, U24 to U23, U21 to U24
Connections:
- CAN1 pad 4: Net-(CAN1-Pin_4) -> +5V
- U21 pad 28: unconnected-(U2-21_A7_RX5_BCLK1-Pad28) -> CAN_STB
- U21 pad 29: /CAN_TX -> CAN_TX
- U21 pad 30: /CAN_RX -> CAN_RX
Routing:
- net Net-(J14-Pin_1): track 37.0 -> 0.00 mm
- net /CAN_RX: track 32.0 -> 0.00 mm
- net ESP_EN: track 30.6 -> 0.00 mm, vias 2 -> 0
- net GND: track 37.0 -> 6.60 mm, vias 12 -> 3
- net /CAN_TX: track 23.1 -> 0.00 mm
- net ESP_TX: track 61.0 -> 38.5 mm, vias 1 -> 0
- net +5V: track 278.2 -> 299.6 mm, vias 2 -> 1
- net U0TXD: track 20.7 -> 0.00 mm, vias 2 -> 0
- net U0RXD: track 20.3 -> 0.00 mm, vias 2 -> 0
- net ESP_RX_OUT: track 18.2 -> 0.00 mm
- net CAN_STB: track 0.00 -> 17.8 mm
- net IO0: track 15.6 -> 0.00 mm
- net BUTTON: track 78.4 -> 63.5 mm, vias 1 -> 2
- net CAN_TX: track 0.00 -> 14.1 mm
- net CAN_LO: track 9.79 -> 22.6 mm
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Other:
- board text added: "BRAIN BOARD V1.4"
- board text added: "CAN"
- board text added: "RX"
- board text added: "TX"
- board text removed: "BOOT"
- board text removed: "CAN VOLT SELECT"
- board text removed: "ENBL"
- board text removed: "ESP32-WROOM-32D"
- board text removed: "MESC BRAIN BOARD V1.2"
- board text removed: "PROG_Rx"
- board text removed: "PROG_Tx"
- board text removed: "Rx"
- board text removed: "Tx"

Commit message: finalization of BB V1.4
Parts:
- added DC_13: 100nF, Capacitor_SMD:C_0603_1608Metric, F.Cu at (51.8, 22.4)
- added U25: SN74LVC14AD, SN74LVC14AD:SOIC127P600X175-14N, F.Cu at (58.8, 25.2)
- moved ESP1 18.1 mm to (70.0, 75.6), turned to 180 degrees
- moved 10k_23 8.17 mm to (87.8, 61.5)
- moved U22 8.17 mm to (83.5, 59.0)
- moved GPIO1 8.17 mm to (66.4, 56.6)
- moved U21 8.17 mm to (72.6, 44.2)
- moved IMU1 8.17 mm to (56.9, 31.6)
- moved 10k_22 8.17 mm to (87.1, 56.5)
- moved C21 8.17 mm to (83.5, 65.7)
- moved CAN1 8.17 mm to (86.3, 74.4)
- moved DC_23 8.17 mm to (83.7, 54.3)
- moved R60_21 8.17 mm to (85.4, 65.7)
- moved TP21 8.17 mm to (81.0, 81.4)
- moved TP22 8.17 mm to (84.8, 81.4)
- moved D21 8.17 mm to (83.3, 69.1)
- moved R60_22 8.17 mm to (81.8, 65.5)
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Connections:
- net INT1 renamed IMU_INT
- C21 pad 1: CAN_CM_BIAS -> Net-(C21-Pad1)
- R60_21 pad 1: CAN_CM_BIAS -> Net-(C21-Pad1)
- R60_22 pad 2: CAN_CM_BIAS -> Net-(C21-Pad1)
- U21 pad 10: RC_Throttle -> RC2
- U21 pad 11: RC_Steering -> RC1
- U21 pad 6: RC_Z -> RC6
- U21 pad 7: RC_Y -> RC5
- U21 pad 8: RC_X -> RC4
- U21 pad 9: RC_Mode -> RC3
- U22 pad 5: CAN_CM_BIAS -> unconnected-(U22-Vref-Pad5)
Routing:
- net RC6: track 0.00 -> 28.3 mm, vias 0 -> 2
- net RC_Z: track 59.9 -> 34.4 mm
- net RC5: track 0.00 -> 23.7 mm, vias 0 -> 2
- net RC_X: track 49.4 -> 28.5 mm, vias 0 -> 1
- net RC_Mode: track 45.7 -> 25.1 mm, vias 0 -> 1
- net RC_Y: track 54.4 -> 36.0 mm, vias 0 -> 1
- net RC1: track 0.00 -> 18.3 mm
- net RC4: track 0.00 -> 17.5 mm
- net RC2: track 0.00 -> 17.3 mm
- net RC3: track 0.00 -> 16.8 mm
- net RC_Throttle: track 37.2 -> 20.9 mm, vias 0 -> 1
- net SPEAKER: track 26.3 -> 10.5 mm, vias 0 -> 2
- net CAN_CM_BIAS: track 11.1 -> 0.00 mm, vias 2 -> 0
- net RC_Steering: track 23.8 -> 13.8 mm
- net LED1: track 5.64 -> 15.0 mm
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Other:
- board text added: "ESP32"
- board text added: "GPIO"
- board text added: "IMU"
- board text removed: "RC Tx/Rx"

Commit message: encoder work
Parts:
- removed the REF** at (96.9, 24.6)
- removed the REF** at (20.4, 23.8)
- removed the REF** at (96.9, 80.2)
- removed the REF** at (20.4, 80.2)
- added REF**: MountingHole_3.2mm_M3, MountingHole:MountingHole_3.2mm_M3, F.Cu at (19.9, 23.8)
- added REF**: MountingHole_3.2mm_M3, MountingHole:MountingHole_3.2mm_M3, F.Cu at (96.5, 23.8)
- added REF**: MountingHole_3.2mm_M3, MountingHole:MountingHole_3.2mm_M3, F.Cu at (96.5, 80.2)
- added REF**: MountingHole_3.2mm_M3, MountingHole:MountingHole_3.2mm_M3, F.Cu at (19.9, 80.2)
- moved J24 3.14 mm to (60.5, 67.8)
- moved 20k_31 1.24 mm to (45.6, 73.6)
- moved C32 1.24 mm to (46.5, 68.7)
- moved C33 1.24 mm to (46.5, 70.9)
- moved D_BLU31 1.24 mm to (47.2, 73.6)
- moved U24 1.24 mm to (52.4, 71.8)
- moved C34 1.08 mm to (57.1, 76.9)
- moved 10k_22 0.43 mm to (87.5, 56.5)
- moved J26 0.38 mm to (51.8, 79.9)
- moved C21 0.13 mm to (83.5, 65.5), turned to 90 degrees
- renumbered 20k_22 to 20k_31, C22 to C31, C23 to C32, C24 to C33, C25 to C34, D_BLU21 to D_BLU31, Q21 to Q1
Routing:
- net +5V: track 302.8 -> 298.3 mm
- net +3.3V: track 32.1 -> 28.9 mm
- net GND: track 7.53 -> 9.00 mm, vias 4 -> 5
- net Net-(C21-Pad1): track 4.87 -> 3.89 mm
- net CAN_TX: track 14.1 -> 15.0 mm
Other:
- board text added: "+"
- board text added: "+3.3V ONLY!"
- board text added: "100nF"
- board text added: "5 mm"
- board text added: "Antenna"
- board text added: "B"
- board text added: "C"
- board text added: "E"
- board text added: "KEEP-OUT ZONE"

Commit message: updated brainboard v1.4
Changed lines of the file:
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@@
 		(tags "SOT TO_SOT_SMD")
 		(property "Reference" "Q1"
-			(at 0.402456 -2.681369 0)
+			(at -0.097544 -3.506369 0)
 			(layer "F.SilkS")
 			(effects
@@
 		(tags "SOIC SO")
 		(property "Reference" "U22"
-			(at 0 0 180)
+			(at 0 0 0)
 			(layer "F.SilkS")
 			(effects
