File: PCBs/brainboardV1.4/MESC_brain_board.kicad_sch (KiCad schematic)
At the start: 16 parts, among them J1 Conn_01x18, J21 Conn_01x07, Q1 my_BC337, U1 TJA1050T/CM,118, U2 Teensy4.0

Commit message: brain board V1.4
Parts:
- removed 10k_1, 10k_8: 10k, Resistor_SMD:R_0603_1608Metric, symbol Device:R
- removed DC_1: 100nF, Capacitor_SMD:C_0603_1608Metric, symbol Device:C
- removed JP1: SolderJumper_3_Open, Jumper:SolderJumper-3_P1.3mm_Open_Pad1.0x1.5mm, symbol Jumper:SolderJumper_3_Open
- removed R_120: 120, Resistor_SMD:R_0603_1608Metric, symbol Device:R
- removed S1: TL3342F160QG, Button_Switch_SMD:SW_SPST_B3SL-1022P, symbol Switch:SW_Push
- removed U1: TJA1050T/CM,118, Package_SO:SOIC-8_3.9x4.9mm_P1.27mm, symbol Interface_CAN_LIN:SN65HVD230
- added 10k_11: 10k, Resistor_SMD:R_0603_1608Metric, symbol Device:R
- added 20k_21: 20k, Resistor_SMD:R_0603_1608Metric, symbol Device:R
- added 5k_21: 5k, Resistor_SMD:R_0603_1608Metric, symbol Device:R
- added DC_12: 100nF, Capacitor_SMD:C_0603_1608Metric, symbol Device:C
- added D_GRN21: LED GRN, LED_SMD:LED_0603_1608Metric, symbol Device:LED
- added D_RED21: LED RED, LED_SMD:LED_0603_1608Metric, symbol Device:LED
- added ESP1: Conn_01x04, Connector_JST:JST_PH_B4B-PH-K_1x04_P2.00mm_Vertical, symbol Connector_Generic:Conn_01x04
- added S21: TL3342F160QG, Button_Switch_SMD:SW_Push_SPST_NO_Alps_SKRK, symbol Switch:SW_Push
- renumbered 1k_1 to 1k_21, DC_2 to DC_21, MESC1 to GPIO1, J21 to IMU1, LS1 to LS21, Q1 to Q21, U2 to U21
Connections:
- net +3.3V: now also 10k_11.2
- net +5V: now also CAN1.4 (Pin_4), ESP1.4 (Pin_4)
- net BUTTON: now also 10k_11.1, DC_12.2, S21.2
- net ESP_RX: now also ESP1.3 (Pin_3)
- net ESP_TX: now also ESP1.2 (Pin_2)
- net GND: now also 20k_21.1, 5k_21.1, DC_12.1, ESP1.1 (Pin_1), S21.1
- net LED1: now also D_RED21.2 (A)
- net LED2: now also D_GRN21.2 (A)
- net CAN_STB: now reaches U21.28 (21_A7_RX5_BCLK1)
- new net: 5k_21.2, D_GRN21.1 (K)
- new net: 20k_21.2, D_RED21.1 (K)
Other:
- removed sheet ESP32
- added sheet CAN Sheet (CAN.kicad_sch)
- note added: "CAN"
- note added: "ESP32"
- note added: "GPIO"
- note added: "IMU"
- note added: "RC_PWM"
- note added: "Remove ESP32 -- export serial to separate module ESPs need to have a clock crystal to transmit Fix CAN to be more bullet proof Bigger / more accessible pushbutton Battery footprint blows How about a "activate" for ESCs?"
- note removed: "3.3V CAN transcievers only"
- note removed: "Force TXD recessive during reset Add a pull-up on TXD (MCU→transceiver TXD input), 4.7k-10k to 5 V."
- note removed: "MP2 SER"
- note removed: "Place 47-100 Ω in series with CANH and CANL, right at the transceiver pins. Limits hot-plug / injection current"
- note removed: "Remove ESP32 -- export serial to separate module ESPs need to have a clock crystal to transmit Fix CAN to be more bullet proof -- add through hole termination resistors -- add decoupling cap at Vcc Bigger / more accessible pushbutton Battery footprint blows How about a "activate" for ESCs?"
- moved on the sheet: 1k_21, DC_21

Commit message: finalization of BB V1.4
Parts:
- added DC_13: 100nF, Capacitor_SMD:C_0603_1608Metric, symbol Device:C
- added U25: SN74LVC14AD, SN74LVC14AD:SOIC127P600X175-14N, symbol SN74LVC14AD:SN74LVC14AD
Connections:
- net +3.3V: now also DC_13.2, U25.14 (VCC)
- net GND: now also DC_13.1, U25.7 (GND)
- net RC_Mode: now also U25.5 (3A); no longer U21.9 (7_RX2_OUT1A)
- net RC_Steering: now also U25.1 (1A); no longer U21.11 (9_OUT1C)
- net RC_Throttle: now also U25.3 (2A); no longer U21.10 (8_TX2_IN1)
- net RC_X: now also U25.9 (4A); no longer U21.8 (6_OUT1D)
- net RC_Y: now also U25.11 (5A); no longer U21.7 (5_IN2)
- net RC_Z: now also U25.13 (6A); no longer U21.6 (4_BCLK2)
- net INT1 renamed IMU_INT
- new net RC1: U21.11 (9_OUT1C), U25.2 (1Y)
- new net RC2: U21.10 (8_TX2_IN1), U25.4 (2Y)
- new net RC3: U21.9 (7_RX2_OUT1A), U25.6 (3Y)
- new net RC4: U21.8 (6_OUT1D), U25.8 (4Y)
- new net RC5: U21.7 (5_IN2), U25.10 (5Y)
- new net RC6: U21.6 (4_BCLK2), U25.12 (6Y)
Other:
- moved on the sheet: 10k_11, 1k_21, 20k_21, 5k_21, DC_12, DC_21, D_GRN21, D_RED21, S21, U21

Commit message: encoder work
Parts:
- renumbered Q21 to Q1
Changed lines of the file:
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@@
 		(on_board yes)
 		(dnp no)
-		(property "Reference" "Q21"
+		(property "Reference" "Q1"
 			(at 63.5 69.8499 0)
 			(effects
@@
 			(project "MESC_brain_board"
 				(path "/8920b97c-b80b-47c5-aaa4-fe68c48cd11a"
-					(reference "Q21")
+					(reference "Q1")
 					(unit 1)
 				)

Commit message: updated brainboard v1.4
Parts:
- D_GRN21: value LED GRN -> APT1608SGC; LCSC C72043 -> APT1608SGC
- D_RED21: LCSC C2286 -> APT1608SURCK
- Q1: value my_BC337 -> SI2302DDS-T1-BE3
- S21: value TL3342F160QG -> TL1015AF160QG; LCSC C318884 -> (none)
Other:
- note added: "Speaker driver • Gate driven low-side logic MOSFET • Drain = speaker node, Source = GND, Gate = control signal • TBD: use a pull-down on gate prevent noise at boot up"
Changed lines of the file:
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@@
 		)
 	)
+	(text "Speaker driver\n• Gate driven low-side logic MOSFET\n• Drain = speaker node, Source = GND, Gate = control signal\n• TBD: use a pull-down on gate prevent noise at boot up"
+		(exclude_from_sim no)
+		(at 43.18 84.074 0)
+		(effects
+			(font
+				(size 1.27 1.27)
+			)
+			(justify left)
+		)
+	)
 	(text "CAN"
 		(exclude_from_sim no)
@@
 			)
 		)
-		(property "Value" "LED GRN"
+		(property "Value" "APT1608SGC"
 			(at 50.8 142.24 0)
 			(effects
@@
 			)
 		)
-		(property "LCSC" "C72043"
+		(property "LCSC" "APT1608SGC"
 			(at 52.07 146.05 0)
 			(effects
@@
 			)
 		)
-		(property "Description" ""
+		(property "Description" "DEV-15583"
 			(at 151.13 55.88 0)
 			(effects
@@
 			)
 		)
-		(property "Value" "my_BC337"
+		(property "Value" "SI2302DDS-T1-BE3"
 			(at 63.754 73.406 0)
 			(effects
@@
 			)
 		)
-		(property "Datasheet" "https://diotec.com/tl_files/diotec/files/pdf/datasheets/bc337.pdf"
+		(property "Datasheet" "https://www.vishay.com/doc?63653"
 			(at 68.58 71.12 0)
 			(effects
@@
 			)
 		)
-		(property "Description" "0.8A Ic, 45V Vce, NPN Transistor, TO-92"
+		(property "Description" "High drive current and efficiency SOT-23 MOSFET"
 			(at 68.58 71.12 0)
 			(effects
@@
 			)
 		)
-		(property "LCSC" "C2286"
+		(property "LCSC" "APT1608SURCK"
 			(at 34.29 146.05 0)
 			(effects
@@
 			)
 		)
-		(property "Value" "TL3342F160QG"
+		(property "Value" "TL1015AF160QG"
 			(at 194.31 36.83 0)
 			(effects
@@
 			)
 		)
-		(property "LCSC" "C318884"
+		(property "LCSC" ""
 			(at 204.47 36.83 0)
 			(effects
