File: PCBs/brainboardV1.4/POWER.kicad_sch (KiCad schematic)
At the start: 16 parts, among them J22 Conn_01x01, J23 Conn_01x01, J24 Conn_01x01, J25 Conn_01x01, U21 LD1117S18TR_SOT223, U24 12_DCDC_5

Commit message: brain board V1.4
Parts:
- removed 20k_1: 20k, Resistor_SMD:R_0603_1608Metric, symbol Device:R
- removed 5k_2: 5k, Resistor_SMD:R_0603_1608Metric, symbol Device:R
- removed D_GRN1: LED GRN, LED_SMD:LED_0603_1608Metric, symbol Device:LED
- removed D_RED1: LED RED, LED_SMD:LED_0603_1608Metric, symbol Device:LED
- renumbered 20k_21 to 20k_22, C21 to C22, C25 to C23, C27 to C24, C23 to C25, J22 to J24, J24 to J26, U24 to U23, U21 to U24

Commit message: encoder work
Parts:
- renumbered 20k_22 to 20k_31, C22 to C31, C23 to C32, C24 to C33, C25 to C34, D_BLU21 to D_BLU31
Changed lines of the file:
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@@
 		(on_board yes)
 		(dnp no)
-		(property "Reference" "20k_22"
+		(property "Reference" "20k_31"
 			(at 199.39 83.185 0)
 			(effects
@@
 			(project "MESC_brain_board"
 				(path "/8920b97c-b80b-47c5-aaa4-fe68c48cd11a/165c0a2c-8484-48b2-be46-c9f57520b95f"
-					(reference "20k_22")
+					(reference "20k_31")
 					(unit 1)
 				)
@@
 		(on_board yes)
 		(dnp no)
-		(property "Reference" "C24"
+		(property "Reference" "C33"
 			(at 162.56 80.01 0)
 			(effects
@@
 			(project "MESC_brain_board"
 				(path "/8920b97c-b80b-47c5-aaa4-fe68c48cd11a/165c0a2c-8484-48b2-be46-c9f57520b95f"
-					(reference "C24")
+					(reference "C33")
 					(unit 1)
 				)
@@
 		(on_board yes)
 		(dnp no)
-		(property "Reference" "C22"
-			(at 127 80.01 0)
+		(property "Reference" "C31"
+			(at 120.904 80.264 0)
 			(effects
 				(font
@@
 			(project "MESC_brain_board"
 				(path "/8920b97c-b80b-47c5-aaa4-fe68c48cd11a/165c0a2c-8484-48b2-be46-c9f57520b95f"
-					(reference "C22")
+					(reference "C31")
 					(unit 1)
 				)
@@
 		(on_board yes)
 		(dnp no)
-		(property "Reference" "C23"
+		(property "Reference" "C32"
 			(at 154.94 80.01 0)
 			(effects
@@
 			(project "MESC_brain_board"
 				(path "/8920b97c-b80b-47c5-aaa4-fe68c48cd11a/165c0a2c-8484-48b2-be46-c9f57520b95f"
-					(reference "C23")
+					(reference "C32")
 					(unit 1)
 				)
@@
 		(on_board yes)
 		(dnp no)
-		(property "Reference" "C25"
+		(property "Reference" "C34"
 			(at 184.785 79.248 0)
 			(effects
@@
 			(project "MESC_brain_board"
 				(path "/8920b97c-b80b-47c5-aaa4-fe68c48cd11a/165c0a2c-8484-48b2-be46-c9f57520b95f"
-					(reference "C25")
+					(reference "C34")
 					(unit 1)
 				)
@@
 		(on_board yes)
 		(dnp no)
-		(property "Reference" "D_BLU21"
+		(property "Reference" "D_BLU31"
 			(at 191.77 69.85 0)
 			(effects
@@
 			(project "MESC_brain_board"
 				(path "/8920b97c-b80b-47c5-aaa4-fe68c48cd11a/165c0a2c-8484-48b2-be46-c9f57520b95f"
-					(reference "D_BLU21")
-					(unit 1)
-				)
+					(reference "D_BLU31")
+					(unit 1)
+				)

Commit message: updated brainboard v1.4
Parts:
- D_BLU31: LCSC C72041 -> APT1608QBC/D
Changed lines of the file:
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@@
 		(dnp no)
 		(property "Reference" "20k_31"
-			(at 199.39 83.185 0)
+			(at 203.708 83.312 0)
 			(effects
 				(font
@@
 			)
 		)
-		(property "LCSC" "C72041"
+		(property "LCSC" "APT1608QBC/D"
 			(at 190.5 76.2 0)
 			(effects
